Commit message: mesh files organized

File: urdf/W3-600B.xacro (robot description, xacro)
@@ -6,22 +6,30 @@
 <link name="base_link">
   <inertial>
-    <origin xyz="-0.011167 0.015936 -0.000013" rpy="0 0 0"/>
-    <mass value="24.024811"/>
-    <inertia ixx="813.7" ixy="4.893" ixz="-0.039975416" iyx="4.893" iyy="2988" iyz="-0.00000417985" izx="-0.039975416" izy="-0.00000417985" izz="2219"/>
-  </inertial>
-  <visual>
-    <origin xyz="0 0 0" rpy="0 0 0"/>
-    <geometry>
-      <mesh filename="package://W3-600B/meshes/base_link.stl" scale="0.001 0.001 0.001"/>
-    </geometry>
-    <material name="silver"/>
-  </visual>
-  <collision>
-    <origin xyz="0 0 0" rpy="0 0 0"/>
-    <geometry>
-      <mesh filename="package://W3-600B/meshes/base_link.stl" scale="0.001 0.001 0.001"/>
-    </geometry>
-  </collision>
-</link>
+    <origin xyz="-0.001608 0.058048 -0.000259" rpy="0 0 0"/>
+    <mass value="69.363439"/>
+    <inertia ixx="3.742" ixy="-0.001876" ixz="0.001144" iyx="-0.001876" iyy="9.426" iyz="0.0002847" izx="0.001144" izy="0.0002847" izz="6.169"/>
+  </inertial>
+  <visual>
+    <origin xyz="0 0 0" rpy="0 0 0"/>
+    <geometry>
+      <mesh filename="package://W3-600B/meshes/base_link_v2.stl" scale="0.001 0.001 0.001"/>
+    </geometry>
+    <material name="silver"/>
+  </visual>
+  <collision>
+    <origin xyz="0 0 0" rpy="0 0 0"/>
+    <geometry>
+      <mesh filename="package://W3-600B/meshes/base_link_v2.stl" scale="0.001 0.001 0.001"/>
+    </geometry>
+  </collision>
+</link>
+<!-- Offset properties -->
+<xacro:property name="caster_support_x_offset" value="0.02"/>
+<xacro:property name="caster_support_y_offset" value="0.0685"/>
+<!-- <xacro:property name="caster_support_z_offset" value="0"/>
+<xacro:property name="caster_wheel_x_offset" value="0"/>
+<xacro:property name="caster_wheel_y_offset" value="0"/>
+<xacro:property name="caster_wheel_z_offset" value="0"/> -->
+<!-- BACK RIGHT CASTER -->
 <link name="caster_wheel_br_1">
   <inertial>
@@ -31,12 +39,12 @@
   </inertial>
   <visual>
-    <origin xyz="-0.309 0.0131 0.248" rpy="0 0 0"/>
-    <geometry>
-      <mesh filename="package://W3-600B/meshes/MANIFOLD_SOLID_BREP_6641.stl" scale="0.001 0.001 0.001"/>
-    </geometry>
-    <material name="silver"/>
-  </visual>
-  <collision>
-    <origin xyz="-0.309 0.0131 0.248" rpy="0 0 0"/>
+    <origin xyz="0 0 0" rpy="0 0 0"/>
+    <geometry>
+      <mesh filename="package://W3-600B/meshes/MANIFOLD_SOLID_BREP_6641.stl" scale="0.001 0.001 0.001"/>
+    </geometry>
+    <material name="silver"/>
+  </visual>
+  <collision>
+    <origin xyz="0 0 0" rpy="0 0 0"/>
     <geometry>
       <mesh filename="package://W3-600B/meshes/MANIFOLD_SOLID_BREP_6641.stl" scale="0.001 0.001 0.001"/>
@@ -51,12 +59,12 @@
   </inertial>
   <visual>
-    <origin xyz="-0.309 0.0131 0.248" rpy="0 0 0"/>
-    <geometry>
-      <mesh filename="package://W3-600B/meshes/MANIFOLD_SOLID_BREP_7274.stl" scale="0.001 0.001 0.001"/>
-    </geometry>
-    <material name="silver"/>
-  </visual>
-  <collision>
-    <origin xyz="-0.309 0.0131 0.248" rpy="0 0 0"/>
+    <origin xyz="0 0 0" rpy="0 0 0"/>
+    <geometry>
+      <mesh filename="package://W3-600B/meshes/MANIFOLD_SOLID_BREP_7274.stl" scale="0.001 0.001 0.001"/>
+    </geometry>
+    <material name="silver"/>
+  </visual>
+  <collision>
+    <origin xyz="0 0 0" rpy="0 0 0"/>
     <geometry>
       <mesh filename="package://W3-600B/meshes/MANIFOLD_SOLID_BREP_7274.stl" scale="0.001 0.001 0.001"/>
@@ -71,17 +79,39 @@
   </inertial>
   <visual>
-    <origin xyz="-0.309 0.0131 0.248" rpy="0 0 0"/>
-    <geometry>
-      <mesh filename="package://W3-600B/meshes/BREP_WITH_VOIDS_6008.stl" scale="0.001 0.001 0.001"/>
-    </geometry>
-    <material name="silver"/>
-  </visual>
-  <collision>
-    <origin xyz="-0.309 0.0131 0.248" rpy="0 0 0"/>
-    <geometry>
-      <mesh filename="package://W3-600B/meshes/BREP_WITH_VOIDS_6008.stl" scale="0.001 0.001 0.001"/>
-    </geometry>
-  </collision>
-</link>
+    <origin xyz="${0 - caster_support_x_offset} ${0 - caster_support_y_offset} 0" rpy="0 0 0"/>
+    <geometry>
+      <mesh filename="package://W3-600B/meshes/BREP_WITH_VOIDS_6008.stl" scale="0.001 0.001 0.001"/>
+    </geometry>
+    <material name="silver"/>
+  </visual>
+  <collision>
+    <origin xyz="${0 - caster_support_x_offset} ${0 - caster_support_y_offset} 0" rpy="0 0 0"/>
+    <geometry>
+      <mesh filename="package://W3-600B/meshes/BREP_WITH_VOIDS_6008.stl" scale="0.001 0.001 0.001"/>
+    </geometry>
+  </collision>
+</link>
+<!-- support joint -->
+<joint name="caster_support_br_joint" type="continuous">
+  <parent link="base_link"/>
+  <child link="caster_support_br"/>
+  <origin xyz="${-0.309 + caster_support_x_offset} ${0.0131 + caster_support_y_offset} 0.248" rpy="0 0 0"/>
+  <axis xyz="0 1 0"/>
+</joint>
+<!-- 1 wheel -->
+<joint name="caster_wheel_br_1_joint" type="continuous">
+  <parent link="caster_support_br"/>
+  <child link="caster_wheel_br_1"/>
+  <origin xyz="${-caster_support_x_offset} ${-caster_support_y_offset} 0" rpy="0 0 0"/>
+  <axis xyz="0 0 1"/>
+</joint>
+<!-- 2 wheel -->
+<joint name="caster_wheel_br_2_joint" type="continuous">
+  <parent link="caster_support_br"/>
+  <child link="caster_wheel_br_2"/>
+  <origin xyz="${-caster_support_x_offset} ${-caster_support_y_offset} 0" rpy="0 0 0"/>
+  <axis xyz="0 0 1"/>
+</joint>
+<!-- BACK LEFT CASTER -->
 <link name="caster_wheel_bl_1">
   <inertial>
@@ -264,24 +294,4 @@
   </collision>
 </link>
-<link name="cameras_support">
-  <inertial>
-    <origin xyz="0 0.079096 -0.050997" rpy="0 0 0"/>
-    <mass value="0.340526"/>
-    <inertia ixx="0.0007119" ixy="-1.748E-19" ixz="0" iyx="-1.748E-19" iyy="0.0003175" iyz="-0.0001125" izx="0" izy="-0.0001125" izz="0.0009268"/>
-  </inertial>
-  <visual>
-    <origin xyz="0 0 0" rpy="0 0 0"/>
-    <geometry>
-      <mesh filename="package://W3-600B/meshes/cameras_support.stl" scale="0.001 0.001 0.001"/>
-    </geometry>
-    <material name="silver"/>
-  </visual>
-  <collision>
-    <origin xyz="0 0 0" rpy="0 0 0"/>
-    <geometry>
-      <mesh filename="package://W3-600B/meshes/cameras_support.stl" scale="0.001 0.001 0.001"/>
-    </geometry>
-  </collision>
-</link>
 <link name="bottom_camera">
   <inertial>
@@ -324,3 +334,103 @@
   </collision>
 </link>
+<link name="back_lidar">
+  <inertial>
+    <origin xyz="-0.42659 0.151334 0" rpy="0 0 0"/>
+    <mass value="1.188679"/>
+    <inertia ixx="0.0007557" ixy="0.000000605351" ixz="-1.051E-17" iyx="0.000000605351" iyy="0.000412" iyz="8.925E-18" izx="-1.051E-17" izy="8.925E-18" izz="0.0007558"/>
+  </inertial>
+  <visual>
+    <origin xyz="0 0 0" rpy="0 0 0"/>
+    <geometry>
+      <mesh filename="package://W3-600B/meshes/lidar.stl" scale="0.001 0.001 0.001"/>
+    </geometry>
+    <material name="silver"/>
+  </visual>
+  <collision>
+    <origin xyz="0 0 0" rpy="0 0 0"/>
+    <geometry>
+      <mesh filename="package://W3-600B/meshes/lidar.stl" scale="0.001 0.001 0.001"/>
+    </geometry>
+  </collision>
+</link>
+<link name="front_lidar">
+  <inertial>
+    <origin xyz="0.423797 0.139017 0.011563" rpy="0 0 0"/>
+    <mass value="0.569677"/>
+    <inertia ixx="0.0009071" ixy="0.000000243534" ixz="0.000014337829" iyx="0.000000243534" iyy="0.0008086" iyz="0.000074824692" izx="0.000014337829" izy="0.000074824692" izz="0.0005095"/>
+  </inertial>
+  <visual>
+    <origin xyz="0.424631 0.1165 0" rpy="0 1.57 0"/>
+    <geometry>
+      <mesh filename="package://W3-600B/meshes/front_lidar.stl" scale="0.001 0.001 0.001"/>
+    </geometry>
+    <material name="silver"/>
+  </visual>
+  <collision>
+    <origin xyz="0.424631 0.1165 0" rpy="0 1.57 0"/>
+    <geometry>
+      <mesh filename="package://W3-600B/meshes/front_lidar.stl" scale="0.001 0.001 0.001"/>
+    </geometry>
+  </collision>
+</link>
+<link name="left_wheel">
+  <inertial>
+    <origin xyz="-0.000216 0.057568 -0.271782" rpy="0 0 0"/>
+    <mass value="9.185826"/>
+    <inertia ixx="0.02957" ixy="-0.000044741546" ixz="0.0001326" iyx="-0.000044741546" iyy="0.03102" iyz="0.000007781675" izx="0.0001326" izy="0.000007781675" izz="0.02782"/>
+  </inertial>
+  <visual>
+    <origin xyz="0 0.0575 -0.131553" rpy="0 0 0"/>
+    <geometry>
+      <mesh filename="package://W3-600B/meshes/left_wheel.stl" scale="0.001 0.001 0.001"/>
+    </geometry>
+    <material name="silver"/>
+  </visual>
+  <collision>
+    <origin xyz="0 0.0575 -0.131553" rpy="0 0 0"/>
+    <geometry>
+      <mesh filename="package://W3-600B/meshes/left_wheel.stl" scale="0.001 0.001 0.001"/>
+    </geometry>
+  </collision>
+</link>
+<link name="right_wheel">
+  <inertial>
+    <origin xyz="0.000216 0.057568 0.271782" rpy="0 0 0"/>
+    <mass value="9.185826"/>
+    <inertia ixx="0.02957" ixy="0.000044741546" ixz="0.0001326" iyx="0.000044741546" iyy="0.03102" iyz="-0.000007781675" izx="0.0001326" izy="-0.000007781675" izz="0.02782"/>
+  </inertial>
+  <visual>
+    <origin xyz="0 0.0575 0.131553" rpy="0 3.14 0"/>
+    <geometry>
+      <mesh filename="package://W3-600B/meshes/right_wheel.stl" scale="0.001 0.001 0.001"/>
+    </geometry>
+    <material name="silver"/>
+  </visual>
+  <collision>
+    <origin xyz="0 0.0575 0.131553" rpy="0 3.14 0"/>
+    <geometry>
+      <mesh filename="package://W3-600B/meshes/right_wheel.stl" scale="0.001 0.001 0.001"/>
+    </geometry>
+  </collision>
+</link>
+<!-- <link name="tray">
+  <inertial>
+    <origin xyz="0.000045 0.218468 -0.0000000000003836" rpy="0 0 0"/>
+    <mass value="58.666118"/>
+    <inertia ixx="2.038" ixy="0.000005613643" ixz="-0.000000000000003583" iyx="0.000005613643" iyy="5.914" iyz="-0.00000000000002564" izx="-0.000000000000003583" izy="-0.00000000000002564" izz="3.878"/>
+  </inertial>
+  <visual>
+    <origin xyz="0 0 0" rpy="0 0 0"/>
+    <geometry>
+      <mesh filename="package://W3-600B/meshes/tray.stl" scale="0.001 0.001 0.001"/>
+    </geometry>
+    <material name="silver"/>
+  </visual>
+  <collision>
+    <origin xyz="0 0 0" rpy="0 0 0"/>
+    <geometry>
+      <mesh filename="package://W3-600B/meshes/tray.stl" scale="0.001 0.001 0.001"/>
+    </geometry>
+  </collision>
+</link> -->
 </robot>
