Commit message: creating macros and joints

File: urdf/W3-600B.urdf (robot description, URDF)
Before this commit: robot W3-600B, 4 links, 0 joints
Links:
- added link back_lidar, mass 1.188679; collision mesh filename=package://W3-600B/meshes/lidar.stl scale=0.001 0.001 0.001; visual mesh filename=package://W3-600B/meshes/lidar.stl scale=0.001 0.001 0.001
- added link bottom_camera, mass 1.384936; collision mesh filename=package://W3-600B/meshes/bottom_camera.stl scale=0.001 0.001 0.001; visual mesh filename=package://W3-600B/meshes/bottom_camera.stl scale=0.001 0.001 0.001
- added link front_lidar, mass 0.569677; collision mesh filename=package://W3-600B/meshes/front_lidar.stl scale=0.001 0.001 0.001; visual mesh filename=package://W3-600B/meshes/front_lidar.stl scale=0.001 0.001 0.001
- added link left_wheel, mass 9.185826; collision mesh filename=package://W3-600B/meshes/left_wheel.stl scale=0.001 0.001 0.001; visual mesh filename=package://W3-600B/meshes/left_wheel.stl scale=0.001 0.001 0.001
- added link right_wheel, mass 9.185826; collision mesh filename=package://W3-600B/meshes/right_wheel.stl scale=0.001 0.001 0.001; visual mesh filename=package://W3-600B/meshes/right_wheel.stl scale=0.001 0.001 0.001
- added link up_camera, mass 1.384936; collision mesh filename=package://W3-600B/meshes/up_camera.stl scale=0.001 0.001 0.001; visual mesh filename=package://W3-600B/meshes/up_camera.stl scale=0.001 0.001 0.001
- link base_link: mass 24.024811 -> 69.363439; geometry collision mesh filename=package://W3-600B/meshes/base_link_v2.stl scale=0.001 0.001 0.001; visual mesh filename=package://W3-600B/meshes/base_link_v2.stl scale=0.001 0.001 0.001
Joints:
- added joint caster_support_br_joint: type continuous, parent base_link, child caster_support_br, origin xyz=-0.289 0.0816 0.248 rpy=0 0 0, axis 0 1 0
- added joint caster_wheel_br_1_joint: type continuous, parent caster_support_br, child caster_wheel_br_1, origin xyz=-0.02 -0.0685 0 rpy=0 0 0, axis 0 0 1
- added joint caster_wheel_br_2_joint: type continuous, parent caster_support_br, child caster_wheel_br_2, origin xyz=-0.02 -0.0685 0 rpy=0 0 0, axis 0 0 1

File: urdf/W3-600B.xacro (robot description, xacro)
@@ -1,7 +1,19 @@
 <?xml version="1.0" ?>
 <robot name="W3-600B" xmlns:xacro="http://www.ros.org/wiki/xacro">
+<!-- Offset properties -->
+<xacro:property name="caster_support_x_offset" value="0.02"/>
+<xacro:property name="caster_support_y_offset" value="0.0685"/>
+<!-- <xacro:property name="caster_support_z_offset" value="0"/>
+<xacro:property name="caster_wheel_x_offset" value="0"/>
+<xacro:property name="caster_wheel_y_offset" value="0"/>
+<xacro:property name="caster_wheel_z_offset" value="0"/> -->
+<!-- Include files -->
 <xacro:include filename="$(find W3-600B)/urdf/materials.xacro" />
 <xacro:include filename="$(find W3-600B)/urdf/W3-600B.trans" />
 <xacro:include filename="$(find W3-600B)/urdf/W3-600B.gazebo" />
+<xacro:include filename="$(find W3-600B)/urdf/caster_wheel.xacro" />
+<xacro:include filename="$(find W3-600B)/urdf/camera.xacro" />
+<xacro:include filename="$(find W3-600B)/urdf/lidar.xacro" />
+<xacro:include filename="$(find W3-600B)/urdf/wheel.xacro" />
 <link name="base_link">
   <inertial>
@@ -24,394 +36,14 @@
   </collision>
 </link>
-<!-- Offset properties -->
-<xacro:property name="caster_support_x_offset" value="0.02"/>
-<xacro:property name="caster_support_y_offset" value="0.0685"/>
-<!-- <xacro:property name="caster_support_z_offset" value="0"/>
-<xacro:property name="caster_wheel_x_offset" value="0"/>
-<xacro:property name="caster_wheel_y_offset" value="0"/>
-<xacro:property name="caster_wheel_z_offset" value="0"/> -->
-<!-- BACK RIGHT CASTER -->
-<link name="caster_wheel_br_1">
-  <inertial>
-    <origin xyz="-0.308999 0.013101 0.26168" rpy="0 0 0"/>
-    <mass value="0.648186"/>
-    <inertia ixx="0.0002538" ixy="-0.000000037013" ixz="6.025E-16" iyx="-0.000000037013" iyy="0.0002526" iyz="7.958E-16" izx="6.025E-16" izy="7.958E-16" izz="0.0004553"/>
-  </inertial>
-  <visual>
-    <origin xyz="0 0 0" rpy="0 0 0"/>
-    <geometry>
-      <mesh filename="package://W3-600B/meshes/MANIFOLD_SOLID_BREP_6641.stl" scale="0.001 0.001 0.001"/>
-    </geometry>
-    <material name="silver"/>
-  </visual>
-  <collision>
-    <origin xyz="0 0 0" rpy="0 0 0"/>
-    <geometry>
-      <mesh filename="package://W3-600B/meshes/MANIFOLD_SOLID_BREP_6641.stl" scale="0.001 0.001 0.001"/>
-    </geometry>
-  </collision>
-</link>
-<link name="caster_wheel_br_2">
-  <inertial>
-    <origin xyz="-0.309 0.013101 0.234319" rpy="0 0 0"/>
-    <mass value="0.648234"/>
-    <inertia ixx="0.0002539" ixy="-0.000000037121" ixz="-0.00000000479" iyx="-0.000000037121" iyy="0.0002526" iyz="-0.00000000012" izx="-0.00000000479" izy="-0.00000000012" izz="0.0004553"/>
-  </inertial>
-  <visual>
-    <origin xyz="0 0 0" rpy="0 0 0"/>
-    <geometry>
-      <mesh filename="package://W3-600B/meshes/MANIFOLD_SOLID_BREP_7274.stl" scale="0.001 0.001 0.001"/>
-    </geometry>
-    <material name="silver"/>
-  </visual>
-  <collision>
-    <origin xyz="0 0 0" rpy="0 0 0"/>
-    <geometry>
-      <mesh filename="package://W3-600B/meshes/MANIFOLD_SOLID_BREP_7274.stl" scale="0.001 0.001 0.001"/>
-    </geometry>
-  </collision>
-</link>
-<link name="caster_support_br">
-  <inertial>
-    <origin xyz="-0.290988 0.064338 0.24807" rpy="0 0 0"/>
-    <mass value="1.304324"/>
-    <inertia ixx="0.001114" ixy="-0.0001204" ixz="0.000001652803" iyx="-0.0001204" iyy="0.001351" iyz="0.000004703024" izx="0.000001652803" izy="0.000004703024" izz="0.001151"/>
-  </inertial>
-  <visual>
-    <origin xyz="${0 - caster_support_x_offset} ${0 - caster_support_y_offset} 0" rpy="0 0 0"/>
-    <geometry>
-      <mesh filename="package://W3-600B/meshes/BREP_WITH_VOIDS_6008.stl" scale="0.001 0.001 0.001"/>
-    </geometry>
-    <material name="silver"/>
-  </visual>
-  <collision>
-    <origin xyz="${0 - caster_support_x_offset} ${0 - caster_support_y_offset} 0" rpy="0 0 0"/>
-    <geometry>
-      <mesh filename="package://W3-600B/meshes/BREP_WITH_VOIDS_6008.stl" scale="0.001 0.001 0.001"/>
-    </geometry>
-  </collision>
-</link>
-<!-- support joint -->
-<joint name="caster_support_br_joint" type="continuous">
-  <parent link="base_link"/>
-  <child link="caster_support_br"/>
-  <origin xyz="${-0.309 + caster_support_x_offset} ${0.0131 + caster_support_y_offset} 0.248" rpy="0 0 0"/>
-  <axis xyz="0 1 0"/>
-</joint>
-<!-- 1 wheel -->
-<joint name="caster_wheel_br_1_joint" type="continuous">
-  <parent link="caster_support_br"/>
-  <child link="caster_wheel_br_1"/>
-  <origin xyz="${-caster_support_x_offset} ${-caster_support_y_offset} 0" rpy="0 0 0"/>
-  <axis xyz="0 0 1"/>
-</joint>
-<!-- 2 wheel -->
-<joint name="caster_wheel_br_2_joint" type="continuous">
-  <parent link="caster_support_br"/>
-  <child link="caster_wheel_br_2"/>
-  <origin xyz="${-caster_support_x_offset} ${-caster_support_y_offset} 0" rpy="0 0 0"/>
-  <axis xyz="0 0 1"/>
-</joint>
-<!-- BACK LEFT CASTER -->
-<link name="caster_wheel_bl_1">
-  <inertial>
-    <origin xyz="-0.30268 0.013101 -0.267999" rpy="0 -1.57 0"/>
-    <mass value="0.648186"/>
-    <inertia ixx="0.0004553" ixy="-7.955E-16" ixz="-6.253E-16" iyx="-7.955E-16" iyy="0.0002526" iyz="-0.000000037013" izx="-6.253E-16" izy="-0.000000037013" izz="0.0002538"/>
-  </inertial>
-  <visual>
-    <origin xyz="-0.289 0.0131 -0.268" rpy="0 -1.57 0"/>
-    <geometry>
-      <mesh filename="package://W3-600B/meshes/MANIFOLD_SOLID_BREP_6641.stl" scale="0.001 0.001 0.001"/>
-    </geometry>
-    <material name="silver"/>
-  </visual>
-  <collision>
-    <origin xyz="-0.289 0.0131 -0.268" rpy="0 -1.57 0"/>
-    <geometry>
-      <mesh filename="package://W3-600B/meshes/MANIFOLD_SOLID_BREP_6641.stl" scale="0.001 0.001 0.001"/>
-    </geometry>
-  </collision>
-</link>
-<link name="caster_wheel_bl_2">
-  <inertial>
-    <origin xyz="-0.275319 0.013101 -0.268" rpy="0 -1.57 0"/>
-    <mass value="0.648234"/>
-    <inertia ixx="0.0004553" ixy="0.00000000012" ixz="0.00000000479" iyx="0.00000000012" iyy="0.0002526" iyz="-0.000000037121" izx="0.00000000479" izy="-0.000000037121" izz="0.0002539"/>
-  </inertial>
-  <visual>
-    <origin xyz="-0.289 0.0131 -0.268" rpy="0 -1.57 0"/>
-    <geometry>
-      <mesh filename="package://W3-600B/meshes/MANIFOLD_SOLID_BREP_7274.stl" scale="0.001 0.001 0.001"/>
-    </geometry>
-    <material name="silver"/>
-  </visual>
-  <collision>
-    <origin xyz="-0.289 0.0131 -0.268" rpy="0 -1.57 0"/>
-    <geometry>
-      <mesh filename="package://W3-600B/meshes/MANIFOLD_SOLID_BREP_7274.stl" scale="0.001 0.001 0.001"/>
-    </geometry>
-  </collision>
-</link>
-<link name="caster_support_bl">
-  <inertial>
-    <origin xyz="-0.28907 0.064338 -0.249988" rpy="0 -1.57 0"/>
-    <mass value="1.304324"/>
-    <inertia ixx="0.001151" ixy="-0.000004703024" ixz="-0.000001652803" iyx="-0.000004703024" iyy="0.001351" iyz="-0.0001204" izx="-0.000001652803" izy="-0.0001204" izz="0.001114"/>
-  </inertial>
-  <visual>
-    <origin xyz="-0.289 0.0131 -0.268" rpy="0 -1.57 0"/>
-    <geometry>
-      <mesh filename="package://W3-600B/meshes/BREP_WITH_VOIDS_6008.stl" scale="0.001 0.001 0.001"/>
-    </geometry>
-    <material name="silver"/>
-  </visual>
-  <collision>
-    <origin xyz="-0.289 0.0131 -0.268" rpy="0 -1.57 0"/>
-    <geometry>
-      <mesh filename="package://W3-600B/meshes/BREP_WITH_VOIDS_6008.stl" scale="0.001 0.001 0.001"/>
-    </geometry>
-  </collision>
-</link>
-<link name="caster_wheel_fr_1">
-  <inertial>
-    <origin xyz="0.32132 0.013101 0.157001" rpy="0 -1.57 0"/>
-    <mass value="0.648186"/>
-    <inertia ixx="0.0004553" ixy="-7.955E-16" ixz="-0.000000000000000631" iyx="-7.955E-16" iyy="0.0002526" iyz="-0.000000037013" izx="-0.000000000000000631" izy="-0.000000037013" izz="0.0002538"/>
-  </inertial>
-  <visual>
-    <origin xyz="0.335 0.0131 0.157" rpy="0 -1.57 0"/>
-    <geometry>
-      <mesh filename="package://W3-600B/meshes/MANIFOLD_SOLID_BREP_6641.stl" scale="0.001 0.001 0.001"/>
-    </geometry>
-    <material name="silver"/>
-  </visual>
-  <collision>
-    <origin xyz="0.335 0.0131 0.157" rpy="0 -1.57 0"/>
-    <geometry>
-      <mesh filename="package://W3-600B/meshes/MANIFOLD_SOLID_BREP_6641.stl" scale="0.001 0.001 0.001"/>
-    </geometry>
-  </collision>
-</link>
-<link name="caster_wheel_fr_2">
-  <inertial>
-    <origin xyz="0.348681 0.013101 0.157" rpy="0 -1.57 0"/>
-    <mass value="0.648234"/>
-    <inertia ixx="0.0004553" ixy="0.00000000012" ixz="0.00000000479" iyx="0.00000000012" iyy="0.0002526" iyz="-0.000000037121" izx="0.00000000479" izy="-0.000000037121" izz="0.0002539"/>
-  </inertial>
-  <visual>
-    <origin xyz="0.335 0.0131 0.157" rpy="0 -1.57 0"/>
-    <geometry>
-      <mesh filename="package://W3-600B/meshes/MANIFOLD_SOLID_BREP_7274.stl" scale="0.001 0.001 0.001"/>
-    </geometry>
-    <material name="silver"/>
-  </visual>
-  <collision>
-    <origin xyz="0.335 0.0131 0.157" rpy="0 -1.57 0"/>
-    <geometry>
-      <mesh filename="package://W3-600B/meshes/MANIFOLD_SOLID_BREP_7274.stl" scale="0.001 0.001 0.001"/>
-    </geometry>
-  </collision>
-</link>
-<link name="caster_support_fr">
-  <inertial>
-    <origin xyz="0.33493 0.064338 0.175012" rpy="0 -1.57 0"/>
-    <mass value="1.304324"/>
-    <inertia ixx="0.001151" ixy="-0.000004703024" ixz="-0.000001652803" iyx="-0.000004703024" iyy="0.001351" iyz="-0.0001204" izx="-0.000001652803" izy="-0.0001204" izz="0.001114"/>
-  </inertial>
-  <visual>
-    <origin xyz="0.335 0.0131 0.157" rpy="0 -1.57 0"/>
-    <geometry>
-      <mesh filename="package://W3-600B/meshes/BREP_WITH_VOIDS_6008.stl" scale="0.001 0.001 0.001"/>
-    </geometry>
-    <material name="silver"/>
-  </visual>
-  <collision>
-    <origin xyz="0.335 0.0131 0.157" rpy="0 -1.57 0"/>
-    <geometry>
-      <mesh filename="package://W3-600B/meshes/BREP_WITH_VOIDS_6008.stl" scale="0.001 0.001 0.001"/>
-    </geometry>
-  </collision>
-</link>
-<link name="caster_wheel_fl_1">
-  <inertial>
-    <origin xyz="0.32132 0.013101 -0.196999" rpy="0 -1.57 0"/>
-    <mass value="0.648186"/>
-    <inertia ixx="0.0004553" ixy="-7.955E-16" ixz="-6.253E-16" iyx="-7.955E-16" iyy="0.0002526" iyz="-0.000000037013" izx="-6.253E-16" izy="-0.000000037013" izz="0.0002538"/>
-  </inertial>
-  <visual>
-    <origin xyz="0.335 0.0131 -0.197" rpy="0 -1.57 0"/>
-    <geometry>
-      <mesh filename="package://W3-600B/meshes/MANIFOLD_SOLID_BREP_6641.stl" scale="0.001 0.001 0.001"/>
-    </geometry>
-    <material name="silver"/>
-  </visual>
-  <collision>
-    <origin xyz="0.335 0.0131 -0.197" rpy="0 -1.57 0"/>
-    <geometry>
-      <mesh filename="package://W3-600B/meshes/MANIFOLD_SOLID_BREP_6641.stl" scale="0.001 0.001 0.001"/>
-    </geometry>
-  </collision>
-</link>
-<link name="caster_wheel_fl_2">
-  <inertial>
-    <origin xyz="0.348681 0.013101 -0.197" rpy="0 -1.57 0"/>
-    <mass value="0.648234"/>
-    <inertia ixx="0.0004553" ixy="0.00000000012" ixz="0.00000000479" iyx="0.00000000012" iyy="0.0002526" iyz="-0.000000037121" izx="0.00000000479" izy="-0.000000037121" izz="0.0002539"/>
-  </inertial>
-  <visual>
-    <origin xyz="0.335 0.0131 -0.197" rpy="0 -1.57 0"/>
-    <geometry>
-      <mesh filename="package://W3-600B/meshes/MANIFOLD_SOLID_BREP_7274.stl" scale="0.001 0.001 0.001"/>
-    </geometry>
-    <material name="silver"/>
-  </visual>
-  <collision>
-    <origin xyz="0.335 0.0131 -0.197" rpy="0 -1.57 0"/>
-    <geometry>
-      <mesh filename="package://W3-600B/meshes/MANIFOLD_SOLID_BREP_7274.stl" scale="0.001 0.001 0.001"/>
-    </geometry>
-  </collision>
-</link>
-<link name="caster_support_fl">
-  <inertial>
-    <origin xyz="0.33493 0.064338 -0.178988" rpy="0 -1.57 0"/>
-    <mass value="1.304324"/>
-    <inertia ixx="0.001151" ixy="-0.000004703024" ixz="-0.000001652803" iyx="-0.000004703024" iyy="0.001351" iyz="-0.0001204" izx="-0.000001652803" izy="-0.0001204" izz="0.001114"/>
-  </inertial>
-  <visual>
-    <origin xyz="0.335 0.0131 -0.197" rpy="0 -1.57 0"/>
-    <geometry>
-      <mesh filename="package://W3-600B/meshes/BREP_WITH_VOIDS_6008.stl" scale="0.001 0.001 0.001"/>
-    </geometry>
-    <material name="silver"/>
-  </visual>
-  <collision>
-    <origin xyz="0.335 0.0131 -0.197" rpy="0 -1.57 0"/>
-    <geometry>
-      <mesh filename="package://W3-600B/meshes/BREP_WITH_VOIDS_6008.stl" scale="0.001 0.001 0.001"/>
-    </geometry>
-  </collision>
-</link>
-<link name="bottom_camera">
-  <inertial>
-    <origin xyz="0 0.076527 0.001765" rpy="0 0 0"/>
-    <mass value="1.384936"/>
-    <inertia ixx="0.00104" ixy="-7.659E-17" ixz="-0.000000000000008721" iyx="-7.659E-17" iyy="0.001219" iyz="-0.000010728685" izx="-0.000000000000008721" izy="-0.000010728685" izz="0.0005682"/>
-  </inertial>
-  <visual>
-    <origin xyz="0 0 0" rpy="0 0 0"/>
-    <geometry>
-      <mesh filename="package://W3-600B/meshes/bottom_camera.stl" scale="0.001 0.001 0.001"/>
-    </geometry>
-    <material name="silver"/>
-  </visual>
-  <collision>
-    <origin xyz="0 0 0" rpy="0 0 0"/>
-    <geometry>
-      <mesh filename="package://W3-600B/meshes/bottom_camera.stl" scale="0.001 0.001 0.001"/>
-    </geometry>
-  </collision>
-</link>
-<link name="up_camera">
-  <inertial>
-    <origin xyz="0 0.148473 0.001765" rpy="0 0 0"/>
-    <mass value="1.384936"/>
-    <inertia ixx="0.00104" ixy="-7.659E-17" ixz="0.000000000000008721" iyx="-7.659E-17" iyy="0.001219" iyz="0.000010728685" izx="0.000000000000008721" izy="0.000010728685" izz="0.0005682"/>
-  </inertial>
-  <visual>
-    <origin xyz="0 0 0" rpy="0 0 0"/>
-    <geometry>
-      <mesh filename="package://W3-600B/meshes/up_camera.stl" scale="0.001 0.001 0.001"/>
-    </geometry>
-    <material name="silver"/>
-  </visual>
-  <collision>
-    <origin xyz="0 0 0" rpy="0 0 0"/>
-    <geometry>
-      <mesh filename="package://W3-600B/meshes/up_camera.stl" scale="0.001 0.001 0.001"/>
-    </geometry>
-  </collision>
-</link>
-<link name="back_lidar">
-  <inertial>
-    <origin xyz="-0.42659 0.151334 0" rpy="0 0 0"/>
-    <mass value="1.188679"/>
-    <inertia ixx="0.0007557" ixy="0.000000605351" ixz="-1.051E-17" iyx="0.000000605351" iyy="0.000412" iyz="8.925E-18" izx="-1.051E-17" izy="8.925E-18" izz="0.0007558"/>
-  </inertial>
-  <visual>
-    <origin xyz="0 0 0" rpy="0 0 0"/>
-    <geometry>
-      <mesh filename="package://W3-600B/meshes/lidar.stl" scale="0.001 0.001 0.001"/>
-    </geometry>
-    <material name="silver"/>
-  </visual>
-  <collision>
-    <origin xyz="0 0 0" rpy="0 0 0"/>
-    <geometry>
-      <mesh filename="package://W3-600B/meshes/lidar.stl" scale="0.001 0.001 0.001"/>
-    </geometry>
-  </collision>
-</link>
-<link name="front_lidar">
-  <inertial>
-    <origin xyz="0.423797 0.139017 0.011563" rpy="0 0 0"/>
-    <mass value="0.569677"/>
-    <inertia ixx="0.0009071" ixy="0.000000243534" ixz="0.000014337829" iyx="0.000000243534" iyy="0.0008086" iyz="0.000074824692" izx="0.000014337829" izy="0.000074824692" izz="0.0005095"/>
-  </inertial>
-  <visual>
-    <origin xyz="0.424631 0.1165 0" rpy="0 1.57 0"/>
-    <geometry>
-      <mesh filename="package://W3-600B/meshes/front_lidar.stl" scale="0.001 0.001 0.001"/>
-    </geometry>
-    <material name="silver"/>
-  </visual>
-  <collision>
-    <origin xyz="0.424631 0.1165 0" rpy="0 1.57 0"/>
-    <geometry>
-      <mesh filename="package://W3-600B/meshes/front_lidar.stl" scale="0.001 0.001 0.001"/>
-    </geometry>
-  </collision>
-</link>
-<link name="left_wheel">
-  <inertial>
-    <origin xyz="-0.000216 0.057568 -0.271782" rpy="0 0 0"/>
-    <mass value="9.185826"/>
-    <inertia ixx="0.02957" ixy="-0.000044741546" ixz="0.0001326" iyx="-0.000044741546" iyy="0.03102" iyz="0.000007781675" izx="0.0001326" izy="0.000007781675" izz="0.02782"/>
-  </inertial>
-  <visual>
-    <origin xyz="0 0.0575 -0.131553" rpy="0 0 0"/>
-    <geometry>
-      <mesh filename="package://W3-600B/meshes/left_wheel.stl" scale="0.001 0.001 0.001"/>
-    </geometry>
-    <material name="silver"/>
-  </visual>
-  <collision>
-    <origin xyz="0 0.0575 -0.131553" rpy="0 0 0"/>
-    <geometry>
-      <mesh filename="package://W3-600B/meshes/left_wheel.stl" scale="0.001 0.001 0.001"/>
-    </geometry>
-  </collision>
-</link>
-<link name="right_wheel">
-  <inertial>
-    <origin xyz="0.000216 0.057568 0.271782" rpy="0 0 0"/>
-    <mass value="9.185826"/>
-    <inertia ixx="0.02957" ixy="0.000044741546" ixz="0.0001326" iyx="0.000044741546" iyy="0.03102" iyz="-0.000007781675" izx="0.0001326" izy="-0.000007781675" izz="0.02782"/>
-  </inertial>
-  <visual>
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