Commit message: changing joint type

File: urdf/wheel.xacro (robot description, xacro)
@@ -29,5 +29,5 @@
             </collision>
         </link>
-        <joint name="${name}_wheel_joint" type="continuous">
+        <joint name="${name}_wheel_joint" type="revolute">
             <parent link="base_link"/>
             <child link="${name}_wheel"/>
