Commit message: fixing 3d robot

File: urdf/camera.xacro (robot description, xacro)
@@ -11,5 +11,5 @@
                 <origin xyz="0 0 0" rpy="0 0 0"/>
                 <geometry>
-                    <mesh filename="package://W3-600B/meshes/${name}_camera.stl" scale="0.001 0.001 0.001"/>
+                    <mesh filename="package://w3_600b/meshes/${name}_camera.stl" scale="0.001 0.001 0.001"/>
                 </geometry>
                 <material name="silver"/>
@@ -18,5 +18,5 @@
                 <origin xyz="0 0 0" rpy="0 0 0"/>
                 <geometry>
-                <mesh filename="package://W3-600B/meshes/bottom_camera.stl" scale="0.001 0.001 0.001"/>
+                <mesh filename="package://w3_600b/meshes/bottom_camera.stl" scale="0.001 0.001 0.001"/>
                 </geometry>
             </collision> -->

File: urdf/caster_wheel.xacro (robot description, xacro)
@@ -12,5 +12,5 @@
                 <origin xyz="0 0 0" rpy="0 0 0"/>
                 <geometry>
-                    <mesh filename="package://W3-600B/meshes/MANIFOLD_SOLID_BREP_6641.stl" scale="0.001 0.001 0.001"/>
+                    <mesh filename="package://w3_600b/meshes/MANIFOLD_SOLID_BREP_6641.stl" scale="0.001 0.001 0.001"/>
                 </geometry>
                 <material name="silver"/>
@@ -19,5 +19,5 @@
                 <origin xyz="0 0 0" rpy="0 0 0"/>
                 <geometry>
-                    <mesh filename="package://W3-600B/meshes/MANIFOLD_SOLID_BREP_6641.stl" scale="0.001 0.001 0.001"/>
+                    <mesh filename="package://w3_600b/meshes/MANIFOLD_SOLID_BREP_6641.stl" scale="0.001 0.001 0.001"/>
                 </geometry>
             </collision>
@@ -32,5 +32,5 @@
                 <origin xyz="0 0 0" rpy="0 0 0"/>
                 <geometry>
-                    <mesh filename="package://W3-600B/meshes/MANIFOLD_SOLID_BREP_7274.stl" scale="0.001 0.001 0.001"/>
+                    <mesh filename="package://w3_600b/meshes/MANIFOLD_SOLID_BREP_7274.stl" scale="0.001 0.001 0.001"/>
                 </geometry>
                 <material name="silver"/>
@@ -39,5 +39,5 @@
                 <origin xyz="0 0 0" rpy="0 0 0"/>
                 <geometry>
-                    <mesh filename="package://W3-600B/meshes/MANIFOLD_SOLID_BREP_7274.stl" scale="0.001 0.001 0.001"/>
+                    <mesh filename="package://w3_600b/meshes/MANIFOLD_SOLID_BREP_7274.stl" scale="0.001 0.001 0.001"/>
                 </geometry>
             </collision>
@@ -52,5 +52,5 @@
                 <origin xyz="${-caster_support_x_offset} ${-caster_support_y_offset} 0" rpy="0 0 0"/>
                 <geometry>
-                    <mesh filename="package://W3-600B/meshes/BREP_WITH_VOIDS_6008.stl" scale="0.001 0.001 0.001"/>
+                    <mesh filename="package://w3_600b/meshes/BREP_WITH_VOIDS_6008.stl" scale="0.001 0.001 0.001"/>
                 </geometry>
                 <material name="silver"/>
@@ -59,5 +59,5 @@
                 <origin xyz="${-caster_support_x_offset} ${-caster_support_y_offset} 0" rpy="0 0 0"/>
                 <geometry>
-                    <mesh filename="package://W3-600B/meshes/BREP_WITH_VOIDS_6008.stl" scale="0.001 0.001 0.001"/>
+                    <mesh filename="package://w3_600b/meshes/BREP_WITH_VOIDS_6008.stl" scale="0.001 0.001 0.001"/>
                 </geometry>
             </collision> -->

File: urdf/lidar.xacro (robot description, xacro)
@@ -17,5 +17,5 @@
                 <origin xyz="${x} ${y} ${z}" rpy="0 ${rotate} 0"/>
                 <geometry>
-                    <mesh filename="package://W3-600B/meshes/${name}_lidar.stl" scale="0.001 0.001 0.001"/>
+                    <mesh filename="package://w3_600b/meshes/${name}_lidar.stl" scale="0.001 0.001 0.001"/>
                 </geometry>
                 <material name="silver"/>
@@ -24,5 +24,5 @@
                 <origin xyz="0.424631 0.1165 0" rpy="0 1.57 0"/>
                 <geometry>
-                    <mesh filename="package://W3-600B/meshes/front_lidar.stl" scale="0.001 0.001 0.001"/>
+                    <mesh filename="package://w3_600b/meshes/front_lidar.stl" scale="0.001 0.001 0.001"/>
                 </geometry>
             </collision> -->

File: urdf/materials.xacro (robot description, xacro)
@@ -1,4 +1,4 @@
 <?xml version="1.0" ?>
-<robot name="W3-600B" xmlns:xacro="http://www.ros.org/wiki/xacro" >
+<robot name="w3_600b" xmlns:xacro="http://www.ros.org/wiki/xacro" >
 <material name="silver">
   <color rgba="0.700 0.700 0.700 1.000"/>

File: urdf/wheel.xacro (robot description, xacro)
@@ -16,14 +16,14 @@
             </inertial>
             <visual>
-                <origin xyz="0 0 0" rpy="0 0 0"/>
+                <origin xyz="0 0 ${wheel_z_offset}" rpy="0 0 0"/>
                 <geometry>
-                    <mesh filename="package://W3-600B/meshes/${name}_wheel.stl" scale="0.001 0.001 0.001"/>
+                    <mesh filename="package://w3_600b/meshes/${name}_wheel.stl" scale="0.001 0.001 0.001"/>
                 </geometry>
                 <material name="silver"/>
             </visual>
             <collision>
-                <origin xyz="0 0 0" rpy="0 0 0"/>
+                <origin xyz="0 0 ${wheel_z_offset}" rpy="0 0 0"/>
                 <geometry>
-                    <mesh filename="package://W3-600B/meshes/${name}_wheel.stl" scale="0.001 0.001 0.001"/>
+                    <mesh filename="package://w3_600b/meshes/${name}_wheel.stl" scale="0.001 0.001 0.001"/>
                 </geometry>
             </collision>
@@ -33,9 +33,10 @@
             <child link="${name}_wheel"/>
             <xacro:if value="${name == 'left'}">
-                <origin xyz="${x} ${y} ${z}" rpy="0 0 0"/>
+                <origin xyz="${x} ${y} ${z-wheel_z_offset}" rpy="0 0 0"/>
             </xacro:if>
             <xacro:if value="${name == 'right'}">
-                <origin xyz="${x} ${y} ${z}" rpy="0 3.14 0"/>
+                <origin xyz="${x} ${y} ${z+wheel_z_offset}" rpy="0 3.14 0"/>
             </xacro:if>
+            <limit effort="22" velocity="${35*2*3.14}" lower="-6.28" upper="6.28"/>
             <axis xyz="0 0 1"/>
         </joint>
