Commit message: organizing files

File: urdf/w3_600b.urdf (robot description, URDF)
Before this commit: robot w3_600b, 10 links, 3 joints
Links:
- removed link bottom_camera
- removed link up_camera
- added link caster_support_bl, mass 1.304324; visual mesh filename=package://w3_600b/meshes/BREP_WITH_VOIDS_6008.stl scale=0.001 0.001 0.001
- added link caster_support_fl, mass 1.304324; visual mesh filename=package://w3_600b/meshes/BREP_WITH_VOIDS_6008.stl scale=0.001 0.001 0.001
- added link caster_support_fr, mass 1.304324; visual mesh filename=package://w3_600b/meshes/BREP_WITH_VOIDS_6008.stl scale=0.001 0.001 0.001
- added link caster_wheel_bl_1, mass 0.648186; collision mesh filename=package://w3_600b/meshes/MANIFOLD_SOLID_BREP_6641.stl scale=0.001 0.001 0.001; visual mesh filename=package://w3_600b/meshes/MANIFOLD_SOLID_BREP_6641.stl scale=0.001 0.001 0.001
- added link caster_wheel_bl_2, mass 0.648234; collision mesh filename=package://w3_600b/meshes/MANIFOLD_SOLID_BREP_7274.stl scale=0.001 0.001 0.001; visual mesh filename=package://w3_600b/meshes/MANIFOLD_SOLID_BREP_7274.stl scale=0.001 0.001 0.001
- added link caster_wheel_fl_1, mass 0.648186; collision mesh filename=package://w3_600b/meshes/MANIFOLD_SOLID_BREP_6641.stl scale=0.001 0.001 0.001; visual mesh filename=package://w3_600b/meshes/MANIFOLD_SOLID_BREP_6641.stl scale=0.001 0.001 0.001
- added link caster_wheel_fl_2, mass 0.648234; collision mesh filename=package://w3_600b/meshes/MANIFOLD_SOLID_BREP_7274.stl scale=0.001 0.001 0.001; visual mesh filename=package://w3_600b/meshes/MANIFOLD_SOLID_BREP_7274.stl scale=0.001 0.001 0.001
- added link caster_wheel_fr_1, mass 0.648186; collision mesh filename=package://w3_600b/meshes/MANIFOLD_SOLID_BREP_6641.stl scale=0.001 0.001 0.001; visual mesh filename=package://w3_600b/meshes/MANIFOLD_SOLID_BREP_6641.stl scale=0.001 0.001 0.001
- added link caster_wheel_fr_2, mass 0.648234; collision mesh filename=package://w3_600b/meshes/MANIFOLD_SOLID_BREP_7274.stl scale=0.001 0.001 0.001; visual mesh filename=package://w3_600b/meshes/MANIFOLD_SOLID_BREP_7274.stl scale=0.001 0.001 0.001
- added link downward_camera; visual mesh filename=package://w3_600b/meshes/downward_camera.stl scale=0.001 0.001 0.001
- added link rotating_base_link
- added link tray, mass 58.666118; collision mesh filename=package://w3_600b/meshes/tray.stl scale=0.001 0.001 0.001; visual mesh filename=package://w3_600b/meshes/tray.stl scale=0.001 0.001 0.001
- added link upward_camera; visual mesh filename=package://w3_600b/meshes/upward_camera.stl scale=0.001 0.001 0.001
- link back_lidar: mass 1.188679 -> None; geometry visual mesh filename=package://w3_600b/meshes/back_lidar.stl scale=0.001 0.001 0.001
- link caster_support_br: geometry visual mesh filename=package://w3_600b/meshes/BREP_WITH_VOIDS_6008.stl scale=0.001 0.001 0.001
- link front_lidar: mass 0.569677 -> None; geometry visual mesh filename=package://w3_600b/meshes/front_lidar.stl scale=0.001 0.001 0.001
Joints:
- added joint caster_support_bl_joint: type continuous, parent base_link, child caster_support_bl, origin xyz=-0.289 0.0816 -0.24800000000000003 rpy=0 0 0, axis 0 1 0
- added joint caster_support_fl_joint: type continuous, parent base_link, child caster_support_fl, origin xyz=0.335 0.0816 -0.17700000000000002 rpy=0 0 0, axis 0 1 0
- added joint caster_support_fr_joint: type continuous, parent base_link, child caster_support_fr, origin xyz=0.335 0.0816 0.177 rpy=0 0 0, axis 0 1 0
- added joint caster_wheel_bl_1_joint: type continuous, parent caster_support_bl, child caster_wheel_bl_1, origin xyz=-0.02 -0.0685 0 rpy=0 0 0, axis 0 0 1
- added joint caster_wheel_bl_2_joint: type continuous, parent caster_support_bl, child caster_wheel_bl_2, origin xyz=-0.02 -0.0685 0 rpy=0 0 0, axis 0 0 1
- added joint caster_wheel_fl_1_joint: type continuous, parent caster_support_fl, child caster_wheel_fl_1, origin xyz=-0.02 -0.0685 0 rpy=0 0 0, axis 0 0 1
- added joint caster_wheel_fl_2_joint: type continuous, parent caster_support_fl, child caster_wheel_fl_2, origin xyz=-0.02 -0.0685 0 rpy=0 0 0, axis 0 0 1
- added joint caster_wheel_fr_1_joint: type continuous, parent caster_support_fr, child caster_wheel_fr_1, origin xyz=-0.02 -0.0685 0 rpy=0 0 0, axis 0 0 1
- added joint caster_wheel_fr_2_joint: type continuous, parent caster_support_fr, child caster_wheel_fr_2, origin xyz=-0.02 -0.0685 0 rpy=0 0 0, axis 0 0 1
- added joint left_wheel_joint: type revolute, parent base_link, child left_wheel, origin xyz=0 0.0575 -0.27875 rpy=0 0 0, axis 0 0 1, limit lower=-6.28 upper=6.28 effort=22 velocity=219.8
- added joint right_wheel_joint: type revolute, parent base_link, child right_wheel, origin xyz=0 0.0575 0.27875 rpy=0 3.14 0, axis 0 0 1, limit lower=-6.28 upper=6.28 effort=22 velocity=219.8
- added joint tray_prismatic_joint: type prismatic, parent rotating_base_link, child tray, origin xyz=0 0 0 rpy=0 0 0, axis 0 1 0, limit lower=0 upper=0.06 effort=5886 velocity=0.013
- added joint tray_revolute_joint: type revolute, parent base_link, child rotating_base_link, origin xyz=0 0 0 rpy=0 0 0, axis 0 1 0, limit lower=-6.28 upper=6.28 effort=5886 velocity=5.233333333333334

File: urdf/w3_600b.xacro (robot description, xacro)
@@ -14,9 +14,10 @@
   <xacro:include filename="$(find w3_600b)/urdf/w3_600b.trans" />
   <xacro:include filename="$(find w3_600b)/urdf/w3_600b.gazebo" />
-  <xacro:include filename="$(find w3_600b)/urdf/caster_wheel.xacro" />
-  <xacro:include filename="$(find w3_600b)/urdf/camera.xacro" />
-  <xacro:include filename="$(find w3_600b)/urdf/lidar.xacro" />
-  <xacro:include filename="$(find w3_600b)/urdf/wheel.xacro" />
-  <xacro:include filename="$(find w3_600b)/urdf/tray.xacro" />
+  <xacro:include filename="$(find w3_600b)/urdf/structure/caster_wheel.xacro" />
+  <xacro:include filename="$(find w3_600b)/urdf/structure/tray.xacro" />
+  <xacro:include filename="$(find w3_600b)/urdf/structure/wheel.xacro" />
+  <xacro:include filename="$(find w3_600b)/urdf/sensors/camera.xacro" />
+  <xacro:include filename="$(find w3_600b)/urdf/sensors/lidar.xacro" />
+  <!-- STRUCTURE -->
   <link name="base_link">
     <inertial>
@@ -50,3 +51,4 @@
   <xacro:wheel name="right" x="0" y="0.0575" z="0.131553"/>
   <xacro:tray/>
+  <!-- CONTROL -->
 </robot>
