Commit message: test

File: urdf/sensors/camera.xacro (robot description, xacro)
@@ -22,4 +22,51 @@
             </collision> -->
         </link>
+        <gazebo reference="${prefix}${name}_color_frame">
+            <sensor name="cam_rgb" type="camera">
+                <pose> 0 0 0 0 0 0 </pose>
+                <visualize>false</visualize>
+                <update_rate>30</update_rate>
+                <camera>
+                    <horizontal_fov>${math.radians(69)}</horizontal_fov>
+                    <vertical_fov>${math.radians(42)}</vertical_fov>
+                    <image>
+                        <format>B8G8R8</format>
+                        <!-- <width>1280</width>
+                        <height>720</height> -->
+                        <width>320</width>
+                        <height>200</height>
+                    </image>
+                    <clip>
+                        <near>0.028</near>
+                        <far>8.0</far>
+                    </clip>
+                </camera>
+                <!-- <camera>
+                    <horizontal_fov>${math.radians(87)}</horizontal_fov>
+                    <vertical_fov>${math.radians(58)}</vertical_fov>
+                    <image>
+                        <format>32FC1</format>
+                        <width>1280</width>
+                        <height>720</height>
+                    </image>
+                    <clip>
+                        <near>0.028</near>
+                        <far>2.0</far>
+                    </clip>
+                    <depth_camera>
+                        <clip>
+                            <near>0.028</near>
+                            <far>2.0</far>
+                        </clip>
+                    </depth_camera>
+                </camera> -->
+                <plugin name="camera_controller_rgb" filename="libgazebo_ros_camera.so">
+                    <ros>
+                        <namespace>/$(arg model_name)/camera_sensor_broadcaster </namespace>
+                    </ros>
+                    <frame_name>${prefix}${name}_color_frame</frame_name>
+                </plugin>
+            </sensor>
+        </gazebo>
     </xacro:macro>
 </robot>

File: urdf/sensors/lidar.xacro (robot description, xacro)
@@ -28,4 +28,52 @@
             </collision> -->
         </link>
+        <gazebo reference="${prefix}${link}">
+            <!-- <material value="Gazebo/Yellow" /> -->
+            <material value="Gazebo/FlatBlack" />
+            <sensor type="ray" name="${prefix}${link}">
+                <pose>0 0 0 0 0 0</pose>
+                <visualize>false</visualize>
+                <update_rate>12.5</update_rate>
+                <ray>
+                    <scan>
+                        <horizontal>
+                            <samples>684</samples>
+                            <resolution>1</resolution>  <!-- has to be 1; actual resolution will be computed from number of samples + min_angle/max_angle -->
+                            <min_angle>-2.35619449615</min_angle>
+                            <max_angle>2.35619449615</max_angle>
+                        </horizontal>
+                    </scan>
+                    <range>
+                        <min>0.05</min>
+                        <max>29.0</max>
+                        <resolution>0.01</resolution>
+                    </range>
+                    <noise>
+                        <type>gaussian</type>
+                        <!-- Noise parameters based on published spec for S300 achieving
+                            "+-29mm" accuracy at range < 3m (~0.01 of the range) at
+                            1 sigma. -->
+                        <mean>0.0</mean>
+                        <stddev>0.01</stddev>
+                    </noise>
+                </ray>
+                <xacro:if value="${gazebo_version == 'classic'}">
+                    <xacro:property name="sensor_name" value="${link.replace('_link','')}"/>
+                    <plugin name="${sensor_name}" filename="libgazebo_ros_ray_sensor.so">
+                        <ros>
+                            <namespace>/$(arg model_name)/lidar_sensor_broadcaster</namespace>
+                            <remapping>${sensor_name}/out:=${sensor_name}/scan</remapping>
+                        </ros>
+                        <output_type>sensor_msgs/LaserScan</output_type>
+                        <frame_name>${prefix}${link}</frame_name>
+                    </plugin>
+                </xacro:if>
+                <xacro:if value="${gazebo_version == 'ignition'}">
+                    <plugin filename="libignition-gazebo-sensors-system.so" name="ignition::gazebo::systems::Sensors">
+                        <render_engine>ogre2</render_engine>
+                    </plugin>
+                </xacro:if>
+            </sensor>
+        </gazebo>
     </xacro:macro>
 </robot>

File: urdf/w3_600b.xacro (robot description, xacro)
@@ -1,4 +1,12 @@
 <?xml version="1.0" ?>
 <robot name="w3_600b" xmlns:xacro="http://www.ros.org/wiki/xacro">
+  <!-- Model properties -->
+  <xacro:property name="model_class" value="robots" />
+  <xacro:property name="model" value="w3_600b" />
+  <xacro:arg name="model_name" default="bot" />
+  <!-- Simulation properties -->
+  <xacro:arg name="gazebo_version" default="classic" />
+  <xacro:property name="gazebo_version" value="$(arg gazebo_version)"/>
+  <coppelia_file filename="$(find w3_600b)/models/${model_class}/${model}/files/CoppeliaSim/w3_600b.ttm"/>
   <!-- Offset properties -->
   <xacro:property name="caster_support_x_offset" value="0.02"/>
@@ -44,11 +52,102 @@
   <xacro:caster_wheel name="fr" x="0.335" y="0.0131" z="0.157"/>
   <xacro:caster_wheel name="fl" x="0.335" y="0.0131" z="-0.197"/>
-  <xacro:camera name="downward"/>
+  <!-- <xacro:camera name="downward"/>
   <xacro:camera name="upward"/>
   <xacro:lidar name="front" x="0.424631" y="0.1165" z="0"/>
-  <xacro:lidar name="back" x="0" y="0" z="0"/>
+  <xacro:lidar name="back" x="0" y="0" z="0"/> -->
   <xacro:wheel name="left" x="0" y="0.0575" z="-0.131553"/>
   <xacro:wheel name="right" x="0" y="0.0575" z="0.131553"/>
   <xacro:tray/>
   <!-- CONTROL -->
+  <xacro:if value="${gazebo_version == 'classic'}">
+    <ros2_control name="GazeboSystem" type="system">
+      <hardware>
+        <plugin>gazebo_ros2_control/GazeboSystem</plugin>
+      </hardware>
+      <!-- <joint name="${prefix}left_wheel_joint"> -->
+      <joint name="left_wheel_joint">
+        <command_interface name="velocity">
+            <param name="min">-10</param>
+            <param name="max">10</param>
+        </command_interface>
+        <state_interface name="position" />
+        <state_interface name="velocity" />
+      </joint>
+      <!-- <joint name="${prefix}right_wheel_joint"> -->
+      <joint name="right_wheel_joint">
+          <command_interface name="velocity">
+              <param name="min">-10</param>
+              <param name="max">10</param>
+          </command_interface>
+          <state_interface name="velocity" />
+          <state_interface name="position" />
+      </joint>
+      <sensor name="imu_sensor">
+        <state_interface name="orientation.x" />
+        <state_interface name="orientation.y" />
+        <state_interface name="orientation.z" />
+        <state_interface name="orientation.w" />
+        <state_interface name="angular_velocity.x" />
+        <state_interface name="angular_velocity.y" />
+        <state_interface name="angular_velocity.z" />
+        <state_interface name="linear_acceleration.x" />
+        <state_interface name="linear_acceleration.y" />
+        <state_interface name="linear_acceleration.z" />
+      </sensor>
+    </ros2_control>
+    <gazebo>
+      <plugin filename="libgazebo_ros2_control.so" name="gazebo_ros2_control">
+        <ros>
+          <namespace>/$(arg model_name)</namespace>
+        </ros>
+        <parameters>$(find w3_600b)/models/${model_class}/${model}/config/$(arg gazebo_version)/${model}_controllers.yaml</parameters>
+      </plugin>
+    </gazebo>
+  </xacro:if>
+  <xacro:if value="${gazebo_version == 'ignition'}">
+    <ros2_control name="IgnitionSystem" type="system">
+      <hardware>
+        <plugin>ign_ros2_control/IgnitionSystem</plugin>
+      </hardware>
+      <!-- <joint name="${prefix}left_wheel_joint"> -->
+      <joint name="left_wheel_joint">
+        <command_interface name="velocity">
+            <param name="min">-10</param>
+            <param name="max">10</param>
+        </command_interface>
+        <state_interface name="position" />
+        <state_interface name="velocity" />
+      </joint>
+      <!-- <joint name="${prefix}right_wheel_joint"> -->
+      <joint name="right_wheel_joint">
+          <command_interface name="velocity">
+              <param name="min">-10</param>
+              <param name="max">10</param>
+          </command_interface>
+          <state_interface name="velocity" />
+          <state_interface name="position" />
+      </joint>
+      <sensor name="imu_sensor">
+        <state_interface name="orientation.x" />
+        <state_interface name="orientation.y" />
+        <state_interface name="orientation.z" />
+        <state_interface name="orientation.w" />
+        <state_interface name="angular_velocity.x" />
+        <state_interface name="angular_velocity.y" />
+        <state_interface name="angular_velocity.z" />
+        <state_interface name="linear_acceleration.x" />
+        <state_interface name="linear_acceleration.y" />
+        <state_interface name="linear_acceleration.z" />
+      </sensor>
+    </ros2_control>
+    <gazebo>
+      <plugin filename="ign_ros2_control-system" name="ign_ros2_control::IgnitionROS2ControlPlugin">
+        <ros>
+          <namespace>/$(arg model_name)</namespace>
+          <remapping>/$(arg model_name)/joint_states:=/joint_state_broadcaster/joint_states</remapping>
+        </ros>
+        <parameters>$(find w3_600b)/models/${model_class}/${model}/config/$(arg gazebo_version)/${model}_controllers.yaml</parameters>
+      </plugin>
+    </gazebo>
+  </xacro:if>
 </robot>
