Commit message: updating model

File: models/robots/w3_600b/urdf/sensors/lidar.xacro (robot description, xacro)
@@ -28,23 +28,23 @@
             </collision> -->
         </link>
-        <gazebo reference="${prefix}${link}">
+        <gazebo reference="${name}_lidar">
             <!-- <material value="Gazebo/Yellow" /> -->
             <material value="Gazebo/FlatBlack" />
-            <sensor type="ray" name="${prefix}${link}">
-                <pose>0 0 0 0 0 0</pose>
+            <sensor type="ray" name="${name}_lidar_sensor">
+                <pose>0.4299 0 0.194 0 0 0</pose>
                 <visualize>false</visualize>
-                <update_rate>12.5</update_rate>
+                <update_rate>30</update_rate>
                 <ray>
                     <scan>
                         <horizontal>
-                            <samples>684</samples>
+                            <samples>1800</samples>
                             <resolution>1</resolution>  <!-- has to be 1; actual resolution will be computed from number of samples + min_angle/max_angle -->
-                            <min_angle>-2.35619449615</min_angle>
-                            <max_angle>2.35619449615</max_angle>
+                            <min_angle>-1.570796</min_angle>
+                            <max_angle>1.570796</max_angle>
                         </horizontal>
                     </scan>
                     <range>
-                        <min>0.05</min>
-                        <max>29.0</max>
+                        <min>0.1</min>
+                        <max>40.0</max>
                         <resolution>0.01</resolution>
                     </range>
@@ -55,9 +55,9 @@
                             1 sigma. -->
                         <mean>0.0</mean>
-                        <stddev>0.01</stddev>
+                        <stddev>0.03</stddev>
                     </noise>
                 </ray>
                 <xacro:if value="${gazebo_version == 'classic'}">
-                    <xacro:property name="sensor_name" value="${link.replace('_link','')}"/>
+                    <xacro:property name="sensor_name" value="${name}_lidar_sensor"/>
                     <plugin name="${sensor_name}" filename="libgazebo_ros_ray_sensor.so">
                         <ros>
@@ -66,5 +66,5 @@
                         </ros>
                         <output_type>sensor_msgs/LaserScan</output_type>
-                        <frame_name>${prefix}${link}</frame_name>
+                        <frame_name>${name}_lidar</frame_name>
                     </plugin>
                 </xacro:if>
