Commit message: updating model

File: models/robots/w3_600b/urdf/sensors/imu.xacro (robot description, xacro)
@@ -13,8 +13,8 @@
     </link>
     <!-- Junta fixa do IMU ao corpo -->
-    <joint name="imu_joint" type="fixed">
+    <joint name="imu_joint" type="continuous">
       <parent link="base_link"/>
       <child link="imu_link"/>
-      <origin xyz="0 0.1 0" rpy="1.57 0 0"/> <!-- posição relativa -->
+      <origin xyz="0.3259 0.17 0.18194" rpy="-1.57 0 0"/> <!-- posição relativa -->
     </joint>
     <gazebo reference="imu_link">

File: models/robots/w3_600b/urdf/w3_600b.urdf (robot description, URDF)
Before this commit: robot w3_600b, 27 links, 26 joints
Joints:
- joint imu_joint: origin xyz=0 0.1 0 rpy=1.57 0 0 -> xyz=0.3259 0.17 0.18194 rpy=-1.57 0 0; type fixed -> continuous
