Commit message: changing package to model

File: models/robots/w3_600b/urdf/sensors/camera.xacro (robot description, xacro)
@@ -11,5 +11,5 @@
                 <origin xyz="0 0 0" rpy="0 0 0"/>
                 <geometry>
-                    <mesh filename="package://sim_models/models/${model_class}/${model}/meshes/${name}_camera.stl" scale="0.001 0.001 0.001"/>
+                    <mesh filename="model://sim_models/models/${model_class}/${model}/meshes/${name}_camera.stl" scale="0.001 0.001 0.001"/>
                 </geometry>
                 <material name="silver"/>
@@ -18,5 +18,5 @@
                 <origin xyz="0 0 0" rpy="0 0 0"/>
                 <geometry>
-                <mesh filename="package://sim_models/models/${model_class}/${model}/meshes/bottom_camera.stl" scale="0.001 0.001 0.001"/>
+                <mesh filename="model://sim_models/models/${model_class}/${model}/meshes/bottom_camera.stl" scale="0.001 0.001 0.001"/>
                 </geometry>
             </collision> -->

File: models/robots/w3_600b/urdf/sensors/imu.xacro (robot description, xacro)
@@ -1,31 +1,26 @@
 <?xml version="1.0"?>
 <robot xmlns:xacro="http://ros.org/wiki/xacro">
-  <!-- If tf_prefix is given, use "frame tf_prefix/imu_frame", else "imu_frame" -->
-  <xacro:arg name="tf_prefix" default="" />
-  <xacro:property name="tf_prefix" value="$(arg tf_prefix)" />
-  <xacro:if value="${tf_prefix == ''}">
-      <xacro:property name="imu_frame" value="imu_frame" />
-  </xacro:if>
-  <xacro:unless value="${tf_prefix == ''}">
-      <xacro:property name="imu_frame" value="$(arg tf_prefix)/imu_frame" />
-  </xacro:unless>
-  <xacro:macro name="imu_gazebo" params="link imu_topic update_rate stdev">
-    <gazebo reference="${link}">
-      <gravity>true</gravity>
+  <xacro:macro name="imu_gazebo" params="">
+    <link name="imu_link">
+      <inertial>
+        <mass value="0.01"/>
+        <origin xyz="0 0 0" rpy="0 0 0"/>
+        <inertia
+          ixx="1e-6" ixy="0.0"  ixz="0.0"
+          iyy="1e-6" iyz="0.0"
+          izz="1e-6"/>
+      </inertial>
+    </link>
+    <!-- Junta fixa do IMU ao corpo -->
+    <joint name="imu_joint" type="fixed">
+      <parent link="base_link"/>
+      <child link="imu_link"/>
+      <origin xyz="0 0.1 0" rpy="1.57 0 0"/> <!-- posição relativa -->
+    </joint>
+    <gazebo reference="imu_link">
       <sensor name="imu_sensor" type="imu">
         <always_on>true</always_on>
-        <update_rate>1000</update_rate>  <!-- this is not the publish rate -->
-        <visualize>true</visualize>
-        <topic>/model/$(arg model_name)/imu_data</topic>
-        <!-- <plugin filename="ignition-gazebo-imu-system" name="gz::sim::systems::Imu">
-          <topicName>${imu_topic}</topicName>
-          <bodyName>${link}</bodyName>
-          <updateRateHZ>${update_rate}</updateRateHZ>  <!- this is the publish rate ->
-          <gaussianNoise>${stdev * stdev}</gaussianNoise>
-          <xyzOffset>0 0 0</xyzOffset>
-          <rpyOffset>0 0 0</rpyOffset>
-          <frameName>${imu_frame}</frameName>  <!- from real MiR ->
-        </plugin> -->
-        <pose>0 0 0 0 0 0</pose>
+        <update_rate>100</update_rate>
+        <!-- <visualize>true</visualize> -->
       </sensor>
     </gazebo>

File: models/robots/w3_600b/urdf/sensors/lidar.xacro (robot description, xacro)
@@ -17,5 +17,5 @@
                 <origin xyz="${x} ${y} ${z}" rpy="0 ${rotate} 0"/>
                 <geometry>
-                    <mesh filename="package://sim_models/models/${model_class}/${model}/meshes/${name}_lidar.stl" scale="0.001 0.001 0.001"/>
+                    <mesh filename="model://sim_models/models/${model_class}/${model}/meshes/${name}_lidar.stl" scale="0.001 0.001 0.001"/>
                 </geometry>
                 <material name="silver"/>
@@ -24,5 +24,5 @@
                 <origin xyz="0.424631 0.1165 0" rpy="0 1.57 0"/>
                 <geometry>
-                    <mesh filename="package://sim_models/models/${model_class}/${model}/meshes/front_lidar.stl" scale="0.001 0.001 0.001"/>
+                    <mesh filename="model://sim_models/models/${model_class}/${model}/meshes/front_lidar.stl" scale="0.001 0.001 0.001"/>
                 </geometry>
             </collision> -->

File: models/robots/w3_600b/urdf/structure/caster_wheel.xacro (robot description, xacro)
@@ -12,5 +12,5 @@
                 <origin xyz="0 0 0" rpy="0 0 0"/>
                 <geometry>
-                    <mesh filename="package://sim_models/models/${model_class}/${model}/meshes/MANIFOLD_SOLID_BREP_6641.stl" scale="0.001 0.001 0.001"/>
+                    <mesh filename="model://sim_models/models/${model_class}/${model}/meshes/MANIFOLD_SOLID_BREP_6641.stl" scale="0.001 0.001 0.001"/>
                 </geometry>
                 <material name="dark_gray"/>
@@ -19,5 +19,5 @@
                 <origin xyz="0 0 0" rpy="0 0 0"/>
                 <geometry>
-                    <mesh filename="package://sim_models/models/${model_class}/${model}/meshes/MANIFOLD_SOLID_BREP_6641.stl" scale="0.001 0.001 0.001"/>
+                    <mesh filename="model://sim_models/models/${model_class}/${model}/meshes/MANIFOLD_SOLID_BREP_6641.stl" scale="0.001 0.001 0.001"/>
                 </geometry>
             </collision>
@@ -32,5 +32,5 @@
                 <origin xyz="0 0 0" rpy="0 0 0"/>
                 <geometry>
-                    <mesh filename="package://sim_models/models/${model_class}/${model}/meshes/MANIFOLD_SOLID_BREP_7274.stl" scale="0.001 0.001 0.001"/>
+                    <mesh filename="model://sim_models/models/${model_class}/${model}/meshes/MANIFOLD_SOLID_BREP_7274.stl" scale="0.001 0.001 0.001"/>
                 </geometry>
                 <material name="dark_gray"/>
@@ -39,5 +39,5 @@
                 <origin xyz="0 0 0" rpy="0 0 0"/>
                 <geometry>
-                    <mesh filename="package://sim_models/models/${model_class}/${model}/meshes/MANIFOLD_SOLID_BREP_7274.stl" scale="0.001 0.001 0.001"/>
+                    <mesh filename="model://sim_models/models/${model_class}/${model}/meshes/MANIFOLD_SOLID_BREP_7274.stl" scale="0.001 0.001 0.001"/>
                 </geometry>
             </collision>
@@ -52,5 +52,5 @@
                 <origin xyz="${-caster_support_x_offset} ${-caster_support_y_offset} 0" rpy="0 0 0"/>
                 <geometry>
-                    <mesh filename="package://sim_models/models/${model_class}/${model}/meshes/BREP_WITH_VOIDS_6008.stl" scale="0.001 0.001 0.001"/>
+                    <mesh filename="model://sim_models/models/${model_class}/${model}/meshes/BREP_WITH_VOIDS_6008.stl" scale="0.001 0.001 0.001"/>
                 </geometry>
                 <material name="silver"/>
@@ -59,5 +59,5 @@
                 <origin xyz="${-caster_support_x_offset} ${-caster_support_y_offset} 0" rpy="0 0 0"/>
                 <geometry>
-                    <mesh filename="package://sim_models/models/${model_class}/${model}/meshes/BREP_WITH_VOIDS_6008.stl" scale="0.001 0.001 0.001"/>
+                    <mesh filename="model://sim_models/models/${model_class}/${model}/meshes/BREP_WITH_VOIDS_6008.stl" scale="0.001 0.001 0.001"/>
                 </geometry>
             </collision> -->

File: models/robots/w3_600b/urdf/structure/tray.xacro (robot description, xacro)
@@ -11,5 +11,5 @@
                 <origin xyz="0 0 0" rpy="0 0 0"/>
                 <geometry>
-                    <mesh filename="package://sim_models/models/${model_class}/${model}/meshes/tray.stl" scale="0.001 0.001 0.001"/>
+                    <mesh filename="model://sim_models/models/${model_class}/${model}/meshes/tray.stl" scale="0.001 0.001 0.001"/>
                 </geometry>
                 <material name="top_gray"/>
@@ -18,5 +18,5 @@
                 <origin xyz="0 0 0" rpy="0 0 0"/>
                 <geometry>
-                    <mesh filename="package://sim_models/models/${model_class}/${model}/meshes/tray.stl" scale="0.001 0.001 0.001"/>
+                    <mesh filename="model://sim_models/models/${model_class}/${model}/meshes/tray.stl" scale="0.001 0.001 0.001"/>
                 </geometry>
             </collision>

File: models/robots/w3_600b/urdf/structure/wheel.xacro (robot description, xacro)
@@ -18,5 +18,5 @@
                 <origin xyz="0 0 ${wheel_z_offset}" rpy="0 0 0"/>
                 <geometry>
-                    <mesh filename="package://sim_models/models/${model_class}/${model}/meshes/${name}_wheel.stl" scale="0.001 0.001 0.001"/>
+                    <mesh filename="model://sim_models/models/${model_class}/${model}/meshes/${name}_wheel.stl" scale="0.001 0.001 0.001"/>
                 </geometry>
                 <material name="dark_gray"/>
@@ -25,5 +25,5 @@
                 <origin xyz="0 0 ${wheel_z_offset}" rpy="0 0 0"/>
                 <geometry>
-                    <mesh filename="package://sim_models/models/${model_class}/${model}/meshes/${name}_wheel.stl" scale="0.001 0.001 0.001"/>
+                    <mesh filename="model://sim_models/models/${model_class}/${model}/meshes/${name}_wheel.stl" scale="0.001 0.001 0.001"/>
                 </geometry>
             </collision>

File: models/robots/w3_600b/urdf/w3_600b.xacro (robot description, xacro)
@@ -24,4 +24,5 @@
   <xacro:include filename="$(find sim_models)/models/${model_class}/${model}/urdf/structure/wheel.xacro" />
   <xacro:include filename="$(find sim_models)/models/${model_class}/${model}/urdf/sensors/camera.xacro" />
+  <xacro:include filename="$(find sim_models)/models/${model_class}/${model}/urdf/sensors/imu.xacro" />
   <xacro:include filename="$(find sim_models)/models/${model_class}/${model}/urdf/sensors/lidar.xacro" />
   <!-- STRUCTURE -->
@@ -36,5 +37,5 @@
       <origin xyz="0 0 0" rpy="0 0 0"/>
       <geometry>
-        <mesh filename="package://sim_models/models/${model_class}/${model}/meshes/base_link_v2.stl" scale="0.001 0.001 0.001"/>
+        <mesh filename="model://sim_models/models/${model_class}/${model}/meshes/base_link_v2.stl" scale="0.001 0.001 0.001"/>
       </geometry>
       <material name="blue_body"/>
@@ -43,5 +44,5 @@
       <origin xyz="0 0 0" rpy="0 0 0"/>
       <geometry>
-        <mesh filename="package://sim_models/models/${model_class}/${model}/meshes/base_link_v2.stl" scale="0.001 0.001 0.001"/>
+        <mesh filename="model://sim_models/models/${model_class}/${model}/meshes/base_link_v2.stl" scale="0.001 0.001 0.001"/>
       </geometry>
     </collision>
@@ -60,4 +61,5 @@
   <xacro:lidar name="front" x="0.424631" y="0.1165" z="0"/>
   <xacro:lidar name="back" x="0" y="0" z="0"/> -->
+  <xacro:imu_gazebo/>
   <xacro:wheel name="left" x="0" y="0.0575" z="-0.131553"/>
   <xacro:wheel name="right" x="0" y="0.0575" z="0.131553"/>
@@ -93,5 +95,5 @@
       <state_interface name="position" />
     </joint>
-    <!-- <sensor name="imu_sensor">
+    <sensor name="imu_sensor">
       <state_interface name="orientation.x" />
       <state_interface name="orientation.y" />
@@ -104,5 +106,5 @@
       <state_interface name="linear_acceleration.y" />
       <state_interface name="linear_acceleration.z" />
-    </sensor> -->
+    </sensor>
   </ros2_control>
   <gazebo>
@@ -118,5 +120,6 @@
       <ros>
         <namespace>$(arg model_name)</namespace>
-        <remapping>/$(arg model_name)/joint_states:=/encoder/joint_states</remapping>
+        <!-- <remapping>/$(arg model_name)/joint_states:=encoders/joint_states</remapping>
+        <remapping>/$(arg model_name)/dynamic_joint_states:=encoders/dynamic_joint_states</remapping> -->
       </ros>
       <parameters>$(find sim_models)/models/${model_class}/${model}/config/$(arg gazebo_version)/${model}_controllers.yaml</parameters>
