Commit message: adding color and lidar sensors

File: models/robots/w3_600b/urdf/sensors/camera.xacro (robot description, xacro)
@@ -11,5 +11,5 @@
                 <origin xyz="0 0 0" rpy="0 0 0"/>
                 <geometry>
-                    <mesh filename="model://sim_models/models/${model_class}/${model}/meshes/${name}_camera.stl" scale="0.001 0.001 0.001"/>
+                    <mesh filename="package://sim_models/models/${model_class}/${model}/meshes/${name}_camera.stl" scale="0.001 0.001 0.001"/>
                 </geometry>
                 <material name="silver"/>
@@ -18,5 +18,5 @@
                 <origin xyz="0 0 0" rpy="0 0 0"/>
                 <geometry>
-                <mesh filename="model://sim_models/models/${model_class}/${model}/meshes/bottom_camera.stl" scale="0.001 0.001 0.001"/>
+                <mesh filename="package://sim_models/models/${model_class}/${model}/meshes/bottom_camera.stl" scale="0.001 0.001 0.001"/>
                 </geometry>
             </collision> -->

File: models/robots/w3_600b/urdf/sensors/lidar.xacro (robot description, xacro)
@@ -1,5 +1,5 @@
 <?xml version="1.0" ?>
 <robot xmlns:xacro="http://www.ros.org/wiki/xacro">
-    <xacro:macro name="lidar" params="name x y z">
+    <xacro:macro name="lidar" params="name">
         <link name="${name}_lidar">
             <!-- <inertial>
@@ -9,29 +9,51 @@
             </inertial> -->
             <visual>
-                <xacro:if value="${name == 'front'}">
-                    <xacro:property name="rotate" value="1.57"/>
-                </xacro:if>
-                <xacro:if value="${name == 'back'}">
-                    <xacro:property name="rotate" value="0"/>
-                </xacro:if>
-                <origin xyz="${x} ${y} ${z}" rpy="0 ${rotate} 0"/>
+                <origin xyz="0 0 0" rpy="0 0 0"/>
                 <geometry>
-                    <mesh filename="model://sim_models/models/${model_class}/${model}/meshes/${name}_lidar.stl" scale="0.001 0.001 0.001"/>
+                    <mesh filename="package://sim_models/models/${model_class}/${model}/meshes/back_lidar.stl" scale="0.001 0.001 0.001"/>
                 </geometry>
                 <material name="silver"/>
             </visual>
             <!-- <collision>
-                <origin xyz="0.424631 0.1165 0" rpy="0 1.57 0"/>
+                <origin xyz="0 0 0" rpy="0 0 0"/>
+                <material name="silver"/>
                 <geometry>
-                    <mesh filename="model://sim_models/models/${model_class}/${model}/meshes/front_lidar.stl" scale="0.001 0.001 0.001"/>
+                    <mesh filename="package://sim_models/models/${model_class}/${model}/meshes/${name}_lidar.stl" scale="0.001 0.001 0.001"/>
                 </geometry>
             </collision> -->
         </link>
         <gazebo reference="${name}_lidar">
+            <material value="Gazebo/DarkGrey" />
+        </gazebo>
+        <joint name="${name}_lidar_mesh_joint" type="fixed">
+            <parent link="base_link"/>
+            <child link="${name}_lidar"/>
+            <xacro:if value="${name == 'front'}">
+                <xacro:property name="rotate" value="3.14"/>
+            </xacro:if>
+            <xacro:if value="${name == 'back'}">
+                <xacro:property name="rotate" value="0"/>
+            </xacro:if>
+            <origin xyz="0 0 0" rpy="0 ${rotate} 0"/>
+        </joint>
+        <link name="${name}_lidar_link">
+        </link>
+        <joint name="${name}_lidar_joint" type="fixed">
+            <parent link="base_link"/>
+            <child link="${name}_lidar_link"/>
+            <xacro:if value="${name == 'front'}">
+                <xacro:property name="k" value="1"/>
+            </xacro:if>
+            <xacro:if value="${name == 'back'}">
+                <xacro:property name="k" value="-1"/>
+            </xacro:if>
+            <origin xyz="${k*0.424631} ${0.1165+0.06} 0" rpy="-1.57 ${k*-1.57} 0"/>
+        </joint>
+        <gazebo reference="${name}_lidar_link">
             <!-- <material value="Gazebo/Yellow" /> -->
-            <material value="Gazebo/FlatBlack" />
-            <sensor type="ray" name="${name}_lidar_sensor">
-                <pose>0.4299 0 0.194 0 0 0</pose>
-                <visualize>false</visualize>
+            <!-- <material value="Gazebo/FlatBlack" /> -->
+            <sensor type="ray" name="${name}">
+                <pose>0 0 0 0 0 0</pose>
+                <!-- <visualize>true</visualize> -->
                 <update_rate>30</update_rate>
                 <ray>
@@ -40,6 +62,6 @@
                             <samples>1800</samples>
                             <resolution>1</resolution>  <!-- has to be 1; actual resolution will be computed from number of samples + min_angle/max_angle -->
-                            <min_angle>-1.570796</min_angle>
-                            <max_angle>1.570796</max_angle>
+                            <min_angle>0</min_angle>
+                            <max_angle>3.1415</max_angle>
                         </horizontal>
                     </scan>
@@ -59,12 +81,11 @@
                 </ray>
                 <xacro:if value="${gazebo_version == 'classic'}">
-                    <xacro:property name="sensor_name" value="${name}_lidar_sensor"/>
-                    <plugin name="${sensor_name}" filename="libgazebo_ros_ray_sensor.so">
+                    <plugin name="${name}" filename="libgazebo_ros_ray_sensor.so">
                         <ros>
-                            <namespace>/$(arg model_name)/lidar_sensor_broadcaster</namespace>
-                            <remapping>${sensor_name}/out:=${sensor_name}/scan</remapping>
+                            <namespace>/$(arg model_name)/lidar</namespace>
+                            <remapping>${name}/out:=${name}/scan</remapping>
                         </ros>
                         <output_type>sensor_msgs/LaserScan</output_type>
-                        <frame_name>${name}_lidar</frame_name>
+                        <frame_name>${name}_lidar_link</frame_name>
                     </plugin>
                 </xacro:if>

File: models/robots/w3_600b/urdf/structure/caster_wheel.xacro (robot description, xacro)
@@ -12,5 +12,5 @@
                 <origin xyz="0 0 0" rpy="0 0 0"/>
                 <geometry>
-                    <mesh filename="model://sim_models/models/${model_class}/${model}/meshes/MANIFOLD_SOLID_BREP_6641.stl" scale="0.001 0.001 0.001"/>
+                    <mesh filename="package://sim_models/models/${model_class}/${model}/meshes/MANIFOLD_SOLID_BREP_6641.stl" scale="0.001 0.001 0.001"/>
                 </geometry>
                 <material name="dark_gray"/>
@@ -19,8 +19,11 @@
                 <origin xyz="0 0 0" rpy="0 0 0"/>
                 <geometry>
-                    <mesh filename="model://sim_models/models/${model_class}/${model}/meshes/MANIFOLD_SOLID_BREP_6641.stl" scale="0.001 0.001 0.001"/>
+                    <mesh filename="package://sim_models/models/${model_class}/${model}/meshes/MANIFOLD_SOLID_BREP_6641.stl" scale="0.001 0.001 0.001"/>
                 </geometry>
             </collision>
         </link>
+        <gazebo reference="caster_wheel_${name}_1">
+            <material value="Gazebo/Orange" />
+        </gazebo>
         <link name="caster_wheel_${name}_2">
             <inertial>
@@ -32,5 +35,5 @@
                 <origin xyz="0 0 0" rpy="0 0 0"/>
                 <geometry>
-                    <mesh filename="model://sim_models/models/${model_class}/${model}/meshes/MANIFOLD_SOLID_BREP_7274.stl" scale="0.001 0.001 0.001"/>
+                    <mesh filename="package://sim_models/models/${model_class}/${model}/meshes/MANIFOLD_SOLID_BREP_7274.stl" scale="0.001 0.001 0.001"/>
                 </geometry>
                 <material name="dark_gray"/>
@@ -39,8 +42,11 @@
                 <origin xyz="0 0 0" rpy="0 0 0"/>
                 <geometry>
-                    <mesh filename="model://sim_models/models/${model_class}/${model}/meshes/MANIFOLD_SOLID_BREP_7274.stl" scale="0.001 0.001 0.001"/>
+                    <mesh filename="package://sim_models/models/${model_class}/${model}/meshes/MANIFOLD_SOLID_BREP_7274.stl" scale="0.001 0.001 0.001"/>
                 </geometry>
             </collision>
         </link>
+        <gazebo reference="caster_wheel_${name}_2">
+            <material value="Gazebo/Orange" />
+        </gazebo>
         <link name="caster_support_${name}">
             <inertial>
@@ -52,5 +58,5 @@
                 <origin xyz="${-caster_support_x_offset} ${-caster_support_y_offset} 0" rpy="0 0 0"/>
                 <geometry>
-                    <mesh filename="model://sim_models/models/${model_class}/${model}/meshes/BREP_WITH_VOIDS_6008.stl" scale="0.001 0.001 0.001"/>
+                    <mesh filename="package://sim_models/models/${model_class}/${model}/meshes/BREP_WITH_VOIDS_6008.stl" scale="0.001 0.001 0.001"/>
                 </geometry>
                 <material name="silver"/>
@@ -59,8 +65,11 @@
                 <origin xyz="${-caster_support_x_offset} ${-caster_support_y_offset} 0" rpy="0 0 0"/>
                 <geometry>
-                    <mesh filename="model://sim_models/models/${model_class}/${model}/meshes/BREP_WITH_VOIDS_6008.stl" scale="0.001 0.001 0.001"/>
+                    <mesh filename="package://sim_models/models/${model_class}/${model}/meshes/BREP_WITH_VOIDS_6008.stl" scale="0.001 0.001 0.001"/>
                 </geometry>
             </collision> -->
         </link>
+        <gazebo reference="caster_support_${name}">
+            <material value="Gazebo/Grey" />
+        </gazebo>
         <!-- support joint -->
         <xacro:if value="${name == 'br'}">

File: models/robots/w3_600b/urdf/structure/tray.xacro (robot description, xacro)
@@ -11,5 +11,5 @@
                 <origin xyz="0 0 0" rpy="0 0 0"/>
                 <geometry>
-                    <mesh filename="model://sim_models/models/${model_class}/${model}/meshes/tray.stl" scale="0.001 0.001 0.001"/>
+                    <mesh filename="package://sim_models/models/${model_class}/${model}/meshes/tray.stl" scale="0.001 0.001 0.001"/>
                 </geometry>
                 <material name="top_gray"/>
@@ -18,8 +18,11 @@
                 <origin xyz="0 0 0" rpy="0 0 0"/>
                 <geometry>
-                    <mesh filename="model://sim_models/models/${model_class}/${model}/meshes/tray.stl" scale="0.001 0.001 0.001"/>
+                    <mesh filename="package://sim_models/models/${model_class}/${model}/meshes/tray.stl" scale="0.001 0.001 0.001"/>
                 </geometry>
             </collision>
         </link>
+        <gazebo reference="tray">
+            <material value="Gazebo/DarkGrey" />
+        </gazebo>
         <link name="rotating_base_link">
             <inertial>

File: models/robots/w3_600b/urdf/structure/wheel.xacro (robot description, xacro)
@@ -18,5 +18,5 @@
                 <origin xyz="0 0 ${wheel_z_offset}" rpy="0 0 0"/>
                 <geometry>
-                    <mesh filename="model://sim_models/models/${model_class}/${model}/meshes/${name}_wheel.stl" scale="0.001 0.001 0.001"/>
+                    <mesh filename="package://sim_models/models/${model_class}/${model}/meshes/${name}_wheel.stl" scale="0.001 0.001 0.001"/>
                 </geometry>
                 <material name="dark_gray"/>
@@ -25,8 +25,11 @@
                 <origin xyz="0 0 ${wheel_z_offset}" rpy="0 0 0"/>
                 <geometry>
-                    <mesh filename="model://sim_models/models/${model_class}/${model}/meshes/${name}_wheel.stl" scale="0.001 0.001 0.001"/>
+                    <mesh filename="package://sim_models/models/${model_class}/${model}/meshes/${name}_wheel.stl" scale="0.001 0.001 0.001"/>
                 </geometry>
             </collision>
         </link>
+        <gazebo reference="${name}_wheel">
+            <material value="Gazebo/DarkGrey" />
+        </gazebo>
         <joint name="${name}_wheel_joint" type="revolute">
             <parent link="base_link"/>

File: models/robots/w3_600b/urdf/w3_600b.xacro (robot description, xacro)
@@ -37,5 +37,5 @@
       <origin xyz="0 0 0" rpy="0 0 0"/>
       <geometry>
-        <mesh filename="model://sim_models/models/${model_class}/${model}/meshes/base_link_v2.stl" scale="0.001 0.001 0.001"/>
+        <mesh filename="package://sim_models/models/${model_class}/${model}/meshes/base_link_v2.stl" scale="0.001 0.001 0.001"/>
       </geometry>
       <material name="blue_body"/>
@@ -44,8 +44,11 @@
       <origin xyz="0 0 0" rpy="0 0 0"/>
       <geometry>
-        <mesh filename="model://sim_models/models/${model_class}/${model}/meshes/base_link_v2.stl" scale="0.001 0.001 0.001"/>
+        <mesh filename="package://sim_models/models/${model_class}/${model}/meshes/base_link_v2.stl" scale="0.001 0.001 0.001"/>
       </geometry>
     </collision>
   </link>
+  <gazebo reference="base_link">
+    <material value="Gazebo/SkyBlue" />
+  </gazebo>
   <joint name="base_to_world" type="fixed">
     <parent link="world_link"/>
@@ -58,7 +61,7 @@
   <xacro:caster_wheel name="fl" x="0.335" y="0.0131" z="-0.197"/>
   <!-- <xacro:camera name="downward"/>
-  <xacro:camera name="upward"/>
-  <xacro:lidar name="front" x="0.424631" y="0.1165" z="0"/>
-  <xacro:lidar name="back" x="0" y="0" z="0"/> -->
+  <xacro:camera name="upward"/> -->
+  <xacro:lidar name="front"/>
+  <xacro:lidar name="back"/>
   <xacro:imu_gazebo/>
   <xacro:wheel name="left" x="0" y="0.0575" z="-0.131553"/>

Commit message: adding cameras

File: models/robots/w3_600b/urdf/sensors/camera.xacro (robot description, xacro)
@@ -11,5 +11,5 @@
                 <origin xyz="0 0 0" rpy="0 0 0"/>
                 <geometry>
-                    <mesh filename="package://sim_models/models/${model_class}/${model}/meshes/${name}_camera.stl" scale="0.001 0.001 0.001"/>
+                    <mesh filename="package://sim_models/models/${model_class}/${model}/meshes/${name}ward_camera.stl" scale="0.001 0.001 0.001"/>
                 </geometry>
                 <material name="silver"/>
@@ -22,48 +22,47 @@
             </collision> -->
         </link>
-        <gazebo reference="${prefix}${name}_color_frame">
-            <sensor name="cam_rgb" type="camera">
+        <gazebo reference="${name}_camera">
+            <material value="Gazebo/Orange" />
+        </gazebo>
+        <joint name="${name}_camera_mesh_joint" type="fixed">
+            <parent link="base_link"/>
+            <child link="${name}_camera"/>
+            <origin xyz="0 0 0" rpy="0 0 0"/>
+        </joint>
+        <link name="${name}_camera_link">
+        </link>
+        <joint name="${name}_camera_joint" type="fixed">
+            <parent link="base_link"/>
+            <child link="${name}_camera_link"/>
+            <xacro:if value="${name == 'down'}">
+                <origin xyz="0 0.05 0" rpy="0 0 -1.57"/>
+            </xacro:if>
+            <xacro:if value="${name == 'up'}">
+                <origin xyz="0 0.175 0" rpy="3.14 0 1.57"/>
+            </xacro:if>
+        </joint>
+        <gazebo reference="${name}_camera_link">
+            <sensor name="${name}_rgb" type="camera">
                 <pose> 0 0 0 0 0 0 </pose>
                 <visualize>false</visualize>
-                <update_rate>30</update_rate>
+                <update_rate>5</update_rate>
                 <camera>
-                    <horizontal_fov>${math.radians(69)}</horizontal_fov>
-                    <vertical_fov>${math.radians(42)}</vertical_fov>
+                    <horizontal_fov>1.047198</horizontal_fov> <!-- 60 degrees -->
+                    <vertical_fov>1.047198</vertical_fov> <!-- 60 degrees -->
                     <image>
                         <format>B8G8R8</format>
-                        <!-- <width>1280</width>
-                        <height>720</height> -->
-                        <width>320</width>
-                        <height>200</height>
+                        <width>128</width>
+                        <height>128</height>
                     </image>
                     <clip>
                         <near>0.028</near>
-                        <far>8.0</far>
+                        <far>0.15</far>
                     </clip>
                 </camera>
-                <!-- <camera>
-                    <horizontal_fov>${math.radians(87)}</horizontal_fov>
-                    <vertical_fov>${math.radians(58)}</vertical_fov>
-                    <image>
-                        <format>32FC1</format>
-                        <width>1280</width>
-                        <height>720</height>
-                    </image>
-                    <clip>
-                        <near>0.028</near>
-                        <far>2.0</far>
-                    </clip>
-                    <depth_camera>
-                        <clip>
-                            <near>0.028</near>
-                            <far>2.0</far>
-                        </clip>
-                    </depth_camera>
-                </camera> -->
-                <plugin name="camera_controller_rgb" filename="libgazebo_ros_camera.so">
+                <plugin name="${name}_rgb" filename="libgazebo_ros_camera.so">
                     <ros>
-                        <namespace>/$(arg model_name)/camera_sensor_broadcaster </namespace>
+                        <namespace>/$(arg model_name)/cam</namespace>
                     </ros>
-                    <frame_name>${prefix}${name}_color_frame</frame_name>
+                    <frame_name>${name}_camera_link</frame_name>
                 </plugin>
             </sensor>

File: models/robots/w3_600b/urdf/w3_600b.xacro (robot description, xacro)
@@ -60,6 +60,6 @@
   <xacro:caster_wheel name="fr" x="0.335" y="0.0131" z="0.157"/>
   <xacro:caster_wheel name="fl" x="0.335" y="0.0131" z="-0.197"/>
-  <!-- <xacro:camera name="downward"/>
-  <xacro:camera name="upward"/> -->
+  <xacro:camera name="down"/>
+  <xacro:camera name="up"/>
   <xacro:lidar name="front"/>
   <xacro:lidar name="back"/>
