Commit message: fixing w3_600b coppelia model

File: models/robots/w3_600b/urdf/sensors/camera.xacro (robot description, xacro)
@@ -11,5 +11,10 @@
                 <origin xyz="0 0 0" rpy="0 0 0"/>
                 <geometry>
-                    <mesh filename="package://sim_models/models/${model_class}/${model}/meshes/${name}ward_camera.stl" scale="0.001 0.001 0.001"/>
+                    <xacro:if value="${simplified_mesh == 1}">
+                        <mesh filename="package://sim_models/models/${model_class}/${model}/meshes/${name}ward_camera_simp.stl" scale="0.001 0.001 0.001"/>
+                    </xacro:if>
+                    <xacro:if value="${simplified_mesh == 0}">
+                        <mesh filename="package://sim_models/models/${model_class}/${model}/meshes/${name}ward_camera.stl" scale="0.001 0.001 0.001"/>
+                    </xacro:if>
                 </geometry>
                 <material name="silver"/>

File: models/robots/w3_600b/urdf/sensors/lidar.xacro (robot description, xacro)
@@ -11,5 +11,10 @@
                 <origin xyz="0 0 0" rpy="0 0 0"/>
                 <geometry>
-                    <mesh filename="package://sim_models/models/${model_class}/${model}/meshes/back_lidar.stl" scale="0.001 0.001 0.001"/>
+                    <xacro:if value="${simplified_mesh == 1}">
+                        <mesh filename="package://sim_models/models/${model_class}/${model}/meshes/back_lidar_simp.stl" scale="0.001 0.001 0.001"/>
+                    </xacro:if>
+                    <xacro:if value="${simplified_mesh == 0}">
+                        <mesh filename="package://sim_models/models/${model_class}/${model}/meshes/back_lidar.stl" scale="0.001 0.001 0.001"/>
+                    </xacro:if>
                 </geometry>
                 <material name="silver"/>

File: models/robots/w3_600b/urdf/structure/caster_wheel.xacro (robot description, xacro)
@@ -16,5 +16,10 @@
                 <origin xyz="0 0 0" rpy="0 0 0"/>
                 <geometry>
-                    <mesh filename="package://sim_models/models/${model_class}/${model}/meshes/MANIFOLD_SOLID_BREP_6641.stl" scale="0.001 0.001 0.001"/>
+                    <xacro:if value="${simplified_mesh == 1}">
+                        <mesh filename="package://sim_models/models/${model_class}/${model}/meshes/MANIFOLD_SOLID_BREP_6641_simp.stl" scale="0.001 0.001 0.001"/>
+                    </xacro:if>
+                    <xacro:if value="${simplified_mesh == 0}">
+                        <mesh filename="package://sim_models/models/${model_class}/${model}/meshes/MANIFOLD_SOLID_BREP_6641.stl" scale="0.001 0.001 0.001"/>
+                    </xacro:if>
                 </geometry>
                 <material name="dark_gray"/>
@@ -39,5 +44,10 @@
                 <origin xyz="0 0 0" rpy="0 0 0"/>
                 <geometry>
-                    <mesh filename="package://sim_models/models/${model_class}/${model}/meshes/MANIFOLD_SOLID_BREP_7274.stl" scale="0.001 0.001 0.001"/>
+                    <xacro:if value="${simplified_mesh == 1}">
+                        <mesh filename="package://sim_models/models/${model_class}/${model}/meshes/MANIFOLD_SOLID_BREP_7274_simp.stl" scale="0.001 0.001 0.001"/>
+                    </xacro:if>
+                    <xacro:if value="${simplified_mesh == 0}">
+                        <mesh filename="package://sim_models/models/${model_class}/${model}/meshes/MANIFOLD_SOLID_BREP_7274.stl" scale="0.001 0.001 0.001"/>
+                    </xacro:if>
                 </geometry>
                 <material name="dark_gray"/>
@@ -62,5 +72,10 @@
                 <origin xyz="${-caster_support_x_offset} ${-caster_support_y_offset} 0" rpy="0 0 0"/>
                 <geometry>
-                    <mesh filename="package://sim_models/models/${model_class}/${model}/meshes/BREP_WITH_VOIDS_6008.stl" scale="0.001 0.001 0.001"/>
+                    <xacro:if value="${simplified_mesh == 1}">
+                        <mesh filename="package://sim_models/models/${model_class}/${model}/meshes/BREP_WITH_VOIDS_6008_simp.stl" scale="0.001 0.001 0.001"/>
+                    </xacro:if>
+                    <xacro:if value="${simplified_mesh == 0}">
+                        <mesh filename="package://sim_models/models/${model_class}/${model}/meshes/BREP_WITH_VOIDS_6008.stl" scale="0.001 0.001 0.001"/>
+                    </xacro:if>
                 </geometry>
                 <material name="silver"/>

File: models/robots/w3_600b/urdf/structure/tray.xacro (robot description, xacro)
@@ -11,5 +11,10 @@
                 <origin xyz="0 -0.218468 0" rpy="0 0 0"/>
                 <geometry>
-                    <mesh filename="package://sim_models/models/${model_class}/${model}/meshes/tray.stl" scale="0.001 0.001 0.001"/>
+                    <xacro:if value="${simplified_mesh == 1}">
+                        <mesh filename="package://sim_models/models/${model_class}/${model}/meshes/tray_simp.stl" scale="0.001 0.001 0.001"/>
+                    </xacro:if>
+                    <xacro:if value="${simplified_mesh == 0}">
+                        <mesh filename="package://sim_models/models/${model_class}/${model}/meshes/tray.stl" scale="0.001 0.001 0.001"/>
+                    </xacro:if>
                 </geometry>
                 <material name="top_gray"/>

File: models/robots/w3_600b/urdf/structure/wheel.xacro (robot description, xacro)
@@ -20,5 +20,10 @@
                 <origin xyz="0 0 ${wheel_z_offset}" rpy="0 0 0"/>
                 <geometry>
-                    <mesh filename="package://sim_models/models/${model_class}/${model}/meshes/${name}_wheel.stl" scale="0.001 0.001 0.001"/>
+                    <xacro:if value="${simplified_mesh == 1}">
+                        <mesh filename="package://sim_models/models/${model_class}/${model}/meshes/${name}_wheel_simp.stl" scale="0.001 0.001 0.001"/>
+                    </xacro:if>
+                    <xacro:if value="${simplified_mesh == 0}">
+                        <mesh filename="package://sim_models/models/${model_class}/${model}/meshes/${name}_wheel.stl" scale="0.001 0.001 0.001"/>
+                    </xacro:if>
                 </geometry>
                 <material name="dark_gray"/>

File: models/robots/w3_600b/urdf/w3_600b.xacro (robot description, xacro)
@@ -5,4 +5,6 @@
   <xacro:property name="model" value="w3_600b" />
   <xacro:arg name="model_name" default="r2d2" />
+  <xacro:arg name="simplified_mesh" default="1" />
+  <xacro:property name="simplified_mesh" value="$(arg simplified_mesh)"/>
   <!-- Simulation properties -->
   <xacro:arg name="gazebo_version" default="classic" />
@@ -37,5 +39,10 @@
       <origin xyz="0 0 0" rpy="0 0 0"/>
       <geometry>
-        <mesh filename="package://sim_models/models/${model_class}/${model}/meshes/base_link_v2.stl" scale="0.001 0.001 0.001"/>
+        <xacro:if value="${simplified_mesh == 1}">
+          <mesh filename="package://sim_models/models/${model_class}/${model}/meshes/base_link_v2_simp.stl" scale="0.001 0.001 0.001"/>
+        </xacro:if>
+        <xacro:if value="${simplified_mesh == 0}">
+          <mesh filename="package://sim_models/models/${model_class}/${model}/meshes/base_link_v2.stl" scale="0.001 0.001 0.001"/>
+        </xacro:if>
       </geometry>
       <material name="blue_body"/>
