Commit message: updating package

File: models/robots/w3_600b/urdf/materials.xacro (robot description, xacro)
@@ -1,6 +1,36 @@
 <?xml version="1.0" ?>
 <robot name="w3_600b" xmlns:xacro="http://www.ros.org/wiki/xacro" >
-<material name="silver">
-  <color rgba="0.700 0.700 0.700 1.000"/>
-</material>
+<!-- Cores para Gazebo e RViz2 -->
+  <xacro:property name="color_blue_body" value="0.2 0.6 0.8 1.0"/>     <!-- azul claro -->
+  <xacro:property name="color_dark_gray" value="0.2 0.2 0.2 1.0"/>     <!-- rodas/cinza escuro -->
+  <xacro:property name="color_top_gray" value="0.6 0.6 0.6 1.0"/>      <!-- tampa metálica -->
+  <xacro:property name="color_led_cyan" value="0.0 1.0 1.0 1.0"/>      <!-- LED azul -->
+  <xacro:property name="color_led_pink" value="1.0 0.4 0.8 1.0"/>      <!-- LED rosa -->
+  <xacro:property name="color_button_green" value="0.0 0.8 0.0 1.0"/>  <!-- botão verde -->
+  <xacro:property name="color_button_red" value="0.8 0.0 0.0 1.0"/>    <!-- botão vermelho -->
+  <!-- Material definitions -->
+  <material name="blue_body">
+    <color rgba="${color_blue_body}"/>
+  </material>
+  <material name="dark_gray">
+    <color rgba="${color_dark_gray}"/>
+  </material>
+  <material name="top_gray">
+    <color rgba="${color_top_gray}"/>
+  </material>
+  <material name="led_cyan">
+    <color rgba="${color_led_cyan}"/>
+  </material>
+  <material name="led_pink">
+    <color rgba="${color_led_pink}"/>
+  </material>
+  <material name="button_green">
+    <color rgba="${color_button_green}"/>
+  </material>
+  <material name="button_red">
+    <color rgba="${color_button_red}"/>
+  </material>
+  <material name="silver">
+    <color rgba="0.700 0.700 0.700 1.000"/>
+  </material>
 </robot>

File: models/robots/w3_600b/urdf/sensors/camera.xacro (robot description, xacro)
@@ -11,5 +11,5 @@
                 <origin xyz="0 0 0" rpy="0 0 0"/>
                 <geometry>
-                    <mesh filename="package://w3_600b/meshes/${name}_camera.stl" scale="0.001 0.001 0.001"/>
+                    <mesh filename="package://sim_models/models/${model_class}/${model}/meshes/${name}_camera.stl" scale="0.001 0.001 0.001"/>
                 </geometry>
                 <material name="silver"/>
@@ -18,5 +18,5 @@
                 <origin xyz="0 0 0" rpy="0 0 0"/>
                 <geometry>
-                <mesh filename="package://w3_600b/meshes/bottom_camera.stl" scale="0.001 0.001 0.001"/>
+                <mesh filename="package://sim_models/models/${model_class}/${model}/meshes/bottom_camera.stl" scale="0.001 0.001 0.001"/>
                 </geometry>
             </collision> -->

File: models/robots/w3_600b/urdf/sensors/lidar.xacro (robot description, xacro)
@@ -17,5 +17,5 @@
                 <origin xyz="${x} ${y} ${z}" rpy="0 ${rotate} 0"/>
                 <geometry>
-                    <mesh filename="package://w3_600b/meshes/${name}_lidar.stl" scale="0.001 0.001 0.001"/>
+                    <mesh filename="package://sim_models/models/${model_class}/${model}/meshes/${name}_lidar.stl" scale="0.001 0.001 0.001"/>
                 </geometry>
                 <material name="silver"/>
@@ -24,5 +24,5 @@
                 <origin xyz="0.424631 0.1165 0" rpy="0 1.57 0"/>
                 <geometry>
-                    <mesh filename="package://w3_600b/meshes/front_lidar.stl" scale="0.001 0.001 0.001"/>
+                    <mesh filename="package://sim_models/models/${model_class}/${model}/meshes/front_lidar.stl" scale="0.001 0.001 0.001"/>
                 </geometry>
             </collision> -->
@@ -69,5 +69,5 @@
                     </plugin>
                 </xacro:if>
-                <xacro:if value="${gazebo_version == 'ignition'}">
+                <xacro:if value="${gazebo_version == 'latest'}">
                     <plugin filename="libignition-gazebo-sensors-system.so" name="ignition::gazebo::systems::Sensors">
                         <render_engine>ogre2</render_engine>

File: models/robots/w3_600b/urdf/structure/caster_wheel.xacro (robot description, xacro)
@@ -12,12 +12,12 @@
                 <origin xyz="0 0 0" rpy="0 0 0"/>
                 <geometry>
-                    <mesh filename="package://w3_600b/meshes/MANIFOLD_SOLID_BREP_6641.stl" scale="0.001 0.001 0.001"/>
+                    <mesh filename="package://sim_models/models/${model_class}/${model}/meshes/MANIFOLD_SOLID_BREP_6641.stl" scale="0.001 0.001 0.001"/>
                 </geometry>
-                <material name="silver"/>
+                <material name="dark_gray"/>
             </visual>
             <collision>
                 <origin xyz="0 0 0" rpy="0 0 0"/>
                 <geometry>
-                    <mesh filename="package://w3_600b/meshes/MANIFOLD_SOLID_BREP_6641.stl" scale="0.001 0.001 0.001"/>
+                    <mesh filename="package://sim_models/models/${model_class}/${model}/meshes/MANIFOLD_SOLID_BREP_6641.stl" scale="0.001 0.001 0.001"/>
                 </geometry>
             </collision>
@@ -32,12 +32,12 @@
                 <origin xyz="0 0 0" rpy="0 0 0"/>
                 <geometry>
-                    <mesh filename="package://w3_600b/meshes/MANIFOLD_SOLID_BREP_7274.stl" scale="0.001 0.001 0.001"/>
+                    <mesh filename="package://sim_models/models/${model_class}/${model}/meshes/MANIFOLD_SOLID_BREP_7274.stl" scale="0.001 0.001 0.001"/>
                 </geometry>
-                <material name="silver"/>
+                <material name="dark_gray"/>
             </visual>
             <collision>
                 <origin xyz="0 0 0" rpy="0 0 0"/>
                 <geometry>
-                    <mesh filename="package://w3_600b/meshes/MANIFOLD_SOLID_BREP_7274.stl" scale="0.001 0.001 0.001"/>
+                    <mesh filename="package://sim_models/models/${model_class}/${model}/meshes/MANIFOLD_SOLID_BREP_7274.stl" scale="0.001 0.001 0.001"/>
                 </geometry>
             </collision>
@@ -52,5 +52,5 @@
                 <origin xyz="${-caster_support_x_offset} ${-caster_support_y_offset} 0" rpy="0 0 0"/>
                 <geometry>
-                    <mesh filename="package://w3_600b/meshes/BREP_WITH_VOIDS_6008.stl" scale="0.001 0.001 0.001"/>
+                    <mesh filename="package://sim_models/models/${model_class}/${model}/meshes/BREP_WITH_VOIDS_6008.stl" scale="0.001 0.001 0.001"/>
                 </geometry>
                 <material name="silver"/>
@@ -59,5 +59,5 @@
                 <origin xyz="${-caster_support_x_offset} ${-caster_support_y_offset} 0" rpy="0 0 0"/>
                 <geometry>
-                    <mesh filename="package://w3_600b/meshes/BREP_WITH_VOIDS_6008.stl" scale="0.001 0.001 0.001"/>
+                    <mesh filename="package://sim_models/models/${model_class}/${model}/meshes/BREP_WITH_VOIDS_6008.stl" scale="0.001 0.001 0.001"/>
                 </geometry>
             </collision> -->

File: models/robots/w3_600b/urdf/structure/tray.xacro (robot description, xacro)
@@ -11,16 +11,22 @@
                 <origin xyz="0 0 0" rpy="0 0 0"/>
                 <geometry>
-                    <mesh filename="package://w3_600b/meshes/tray.stl" scale="0.001 0.001 0.001"/>
+                    <mesh filename="package://sim_models/models/${model_class}/${model}/meshes/tray.stl" scale="0.001 0.001 0.001"/>
                 </geometry>
-                <material name="silver"/>
+                <material name="top_gray"/>
             </visual>
             <collision>
                 <origin xyz="0 0 0" rpy="0 0 0"/>
                 <geometry>
-                    <mesh filename="package://w3_600b/meshes/tray.stl" scale="0.001 0.001 0.001"/>
+                    <mesh filename="package://sim_models/models/${model_class}/${model}/meshes/tray.stl" scale="0.001 0.001 0.001"/>
                 </geometry>
             </collision>
         </link>
-        <link name="rotating_base_link" />
+        <link name="rotating_base_link">
+            <inertial>
+                <origin xyz="0.000045 0.218468 -0.0000000000003836" rpy="0 0 0"/>
+                <mass value="58.666118"/>
+                <inertia ixx="2.038" ixy="0.000005613643" ixz="-0.000000000000003583" iyx="0.000005613643" iyy="5.914" iyz="-0.00000000000002564" izx="-0.000000000000003583" izy="-0.00000000000002564" izz="3.878"/>
+            </inertial>
+        </link>
         <joint name="tray_revolute_joint" type="revolute">
             <parent link="base_link"/>

File: models/robots/w3_600b/urdf/structure/wheel.xacro (robot description, xacro)
@@ -18,12 +18,12 @@
                 <origin xyz="0 0 ${wheel_z_offset}" rpy="0 0 0"/>
                 <geometry>
-                    <mesh filename="package://w3_600b/meshes/${name}_wheel.stl" scale="0.001 0.001 0.001"/>
+                    <mesh filename="package://sim_models/models/${model_class}/${model}/meshes/${name}_wheel.stl" scale="0.001 0.001 0.001"/>
                 </geometry>
-                <material name="silver"/>
+                <material name="dark_gray"/>
             </visual>
             <collision>
                 <origin xyz="0 0 ${wheel_z_offset}" rpy="0 0 0"/>
                 <geometry>
-                    <mesh filename="package://w3_600b/meshes/${name}_wheel.stl" scale="0.001 0.001 0.001"/>
+                    <mesh filename="package://sim_models/models/${model_class}/${model}/meshes/${name}_wheel.stl" scale="0.001 0.001 0.001"/>
                 </geometry>
             </collision>

File: models/robots/w3_600b/urdf/w3_600b.xacro (robot description, xacro)
@@ -8,5 +8,5 @@
   <xacro:arg name="gazebo_version" default="classic" />
   <xacro:property name="gazebo_version" value="$(arg gazebo_version)"/>
-  <coppelia_file filename="$(find w3_600b)/models/${model_class}/${model}/files/CoppeliaSim/w3_600b.ttm"/>
+  <coppelia_file filename="$(find sim_models)/models/${model_class}/${model}/files/CoppeliaSim/w3_600b.ttm"/>
   <!-- Offset properties -->
   <xacro:property name="caster_support_x_offset" value="0.02"/>
@@ -19,13 +19,12 @@
   <xacro:property name="tray_y_offset" value="0.21150"/>
   <!-- Include files -->
-  <xacro:include filename="$(find w3_600b)/urdf/materials.xacro" />
-  <xacro:include filename="$(find w3_600b)/urdf/w3_600b.trans" />
-  <xacro:include filename="$(find w3_600b)/urdf/w3_600b.gazebo" />
-  <xacro:include filename="$(find w3_600b)/urdf/structure/caster_wheel.xacro" />
-  <xacro:include filename="$(find w3_600b)/urdf/structure/tray.xacro" />
-  <xacro:include filename="$(find w3_600b)/urdf/structure/wheel.xacro" />
-  <xacro:include filename="$(find w3_600b)/urdf/sensors/camera.xacro" />
-  <xacro:include filename="$(find w3_600b)/urdf/sensors/lidar.xacro" />
+  <xacro:include filename="$(find sim_models)/models/${model_class}/${model}/urdf/materials.xacro" />
+  <xacro:include filename="$(find sim_models)/models/${model_class}/${model}/urdf/structure/caster_wheel.xacro" />
+  <xacro:include filename="$(find sim_models)/models/${model_class}/${model}/urdf/structure/tray.xacro" />
+  <xacro:include filename="$(find sim_models)/models/${model_class}/${model}/urdf/structure/wheel.xacro" />
+  <xacro:include filename="$(find sim_models)/models/${model_class}/${model}/urdf/sensors/camera.xacro" />
+  <xacro:include filename="$(find sim_models)/models/${model_class}/${model}/urdf/sensors/lidar.xacro" />
   <!-- STRUCTURE -->
+  <link name="world_link"/>
   <link name="base_link">
     <inertial>
@@ -37,15 +36,20 @@
       <origin xyz="0 0 0" rpy="0 0 0"/>
       <geometry>
-        <mesh filename="package://w3_600b/meshes/base_link_v2.stl" scale="0.001 0.001 0.001"/>
+        <mesh filename="package://sim_models/models/${model_class}/${model}/meshes/base_link_v2.stl" scale="0.001 0.001 0.001"/>
       </geometry>
-      <material name="silver"/>
+      <material name="blue_body"/>
     </visual>
     <collision>
       <origin xyz="0 0 0" rpy="0 0 0"/>
       <geometry>
-        <mesh filename="package://w3_600b/meshes/base_link_v2.stl" scale="0.001 0.001 0.001"/>
+        <mesh filename="package://sim_models/models/${model_class}/${model}/meshes/base_link_v2.stl" scale="0.001 0.001 0.001"/>
       </geometry>
     </collision>
   </link>
+  <joint name="base_to_world" type="fixed">
+    <parent link="world_link"/>
+    <child link="base_link"/>
+    <origin xyz="0 0 0" rpy="1.57 0 0"/>
+  </joint>
   <xacro:caster_wheel name="br" x="-0.309" y="0.0131" z="0.248"/>
   <xacro:caster_wheel name="bl" x="-0.289" y="0.0131" z="-0.268"/>
@@ -101,14 +105,13 @@
           <namespace>/$(arg model_name)</namespace>
         </ros>
-        <parameters>$(find w3_600b)/models/${model_class}/${model}/config/$(arg gazebo_version)/${model}_controllers.yaml</parameters>
+        <parameters>$(find sim_models)/models/${model_class}/${model}/config/$(arg gazebo_version)/${model}_controllers.yaml</parameters>
       </plugin>
     </gazebo>
   </xacro:if>
-  <xacro:if value="${gazebo_version == 'ignition'}">
-    <ros2_control name="IgnitionSystem" type="system">
+  <xacro:if value="${gazebo_version == 'latest'}">
+    <ros2_control name="GazeboSimSystem" type="system">
       <hardware>
-        <plugin>ign_ros2_control/IgnitionSystem</plugin>
+        <plugin>gz_ros2_control/GazeboSimSystem</plugin>
       </hardware>
-      <!-- <joint name="${prefix}left_wheel_joint"> -->
       <joint name="left_wheel_joint">
         <command_interface name="velocity">
@@ -119,5 +122,4 @@
         <state_interface name="velocity" />
       </joint>
-      <!-- <joint name="${prefix}right_wheel_joint"> -->
       <joint name="right_wheel_joint">
           <command_interface name="velocity">
@@ -128,5 +130,5 @@
           <state_interface name="position" />
       </joint>
-      <sensor name="imu_sensor">
+      <!-- <sensor name="imu_sensor">
         <state_interface name="orientation.x" />
         <state_interface name="orientation.y" />
@@ -139,13 +141,13 @@
         <state_interface name="linear_acceleration.y" />
         <state_interface name="linear_acceleration.z" />
-      </sensor>
+      </sensor> -->
     </ros2_control>
     <gazebo>
-      <plugin filename="ign_ros2_control-system" name="ign_ros2_control::IgnitionROS2ControlPlugin">
+      <plugin filename="gz_ros2_control-system" name="gz_ros2_control::GazeboSimROS2ControlPlugin">
         <ros>
           <namespace>/$(arg model_name)</namespace>
-          <remapping>/$(arg model_name)/joint_states:=/joint_state_broadcaster/joint_states</remapping>
+          <!-- <remapping>/$(arg model_name)/joint_states:=/joint_state_broadcaster/joint_states</remapping> -->
         </ros>
-        <parameters>$(find w3_600b)/models/${model_class}/${model}/config/$(arg gazebo_version)/${model}_controllers.yaml</parameters>
+        <parameters>$(find sim_models)/models/${model_class}/${model}/config/$(arg gazebo_version)/${model}_controllers.yaml</parameters>
       </plugin>
     </gazebo>
