Commit message: gazebo test

File: models/robots/w3_600b/urdf/w3_600b.xacro (robot description, xacro)
@@ -65,27 +65,19 @@
   <!-- CONTROL -->
   <xacro:if value="${gazebo_version == 'classic'}">
-    <ros2_control name="GazeboSystem" type="system">
+    <ros2_control name="TestSystem" type="system">
       <hardware>
         <plugin>gazebo_ros2_control/GazeboSystem</plugin>
       </hardware>
-      <!-- <joint name="${prefix}left_wheel_joint"> -->
       <joint name="left_wheel_joint">
-        <command_interface name="velocity">
-            <param name="min">-10</param>
-            <param name="max">10</param>
-        </command_interface>
+        <command_interface name="velocity"/>
         <state_interface name="position" />
         <state_interface name="velocity" />
       </joint>
-      <!-- <joint name="${prefix}right_wheel_joint"> -->
       <joint name="right_wheel_joint">
-          <command_interface name="velocity">
-              <param name="min">-10</param>
-              <param name="max">10</param>
-          </command_interface>
+          <command_interface name="velocity"/>
           <state_interface name="velocity" />
           <state_interface name="position" />
       </joint>
-      <sensor name="imu_sensor">
+      <!-- <sensor name="imu_sensor">
         <state_interface name="orientation.x" />
         <state_interface name="orientation.y" />
@@ -98,5 +90,5 @@
         <state_interface name="linear_acceleration.y" />
         <state_interface name="linear_acceleration.z" />
-      </sensor>
+      </sensor> -->
     </ros2_control>
     <gazebo>
