Commit message: adding tray controll

File: models/robots/w3_600b/urdf/structure/tray.xacro (robot description, xacro)
@@ -35,4 +35,5 @@
             <axis xyz="0 1 0"/>
             <limit effort="5886" velocity="${300*(3.14/180)}" lower="-6.28" upper="6.28"/>
+            <dynamics damping="0.5" friction="0.1"/>
         </joint>
         <joint name="tray_prismatic_joint" type="prismatic">

File: models/robots/w3_600b/urdf/w3_600b.xacro (robot description, xacro)
@@ -64,79 +64,62 @@
   <xacro:tray/>
   <!-- CONTROL -->
-  <xacro:if value="${gazebo_version == 'classic'}">
-    <ros2_control name="GazeboSystem" type="system">
-      <hardware>
+  <ros2_control name="GazeboSystem" type="system">
+    <hardware>
+      <xacro:if value="${gazebo_version == 'classic'}">
         <plugin>gazebo_ros2_control/GazeboSystem</plugin>
-      </hardware>
-      <joint name="left_wheel_joint">
+      </xacro:if>
+      <xacro:if value="${gazebo_version == 'latest'}">
+        <plugin>gz_ros2_control/GazeboSimSystem</plugin>
+      </xacro:if>
+    </hardware>
+    <joint name="left_wheel_joint">
+      <command_interface name="velocity"/>
+      <state_interface name="position" />
+      <state_interface name="velocity" />
+    </joint>
+    <joint name="right_wheel_joint">
         <command_interface name="velocity"/>
+        <state_interface name="velocity" />
         <state_interface name="position" />
-        <state_interface name="velocity" />
-      </joint>
-      <joint name="right_wheel_joint">
-          <command_interface name="velocity"/>
-          <state_interface name="velocity" />
-          <state_interface name="position" />
-      </joint>
-      <!-- <sensor name="imu_sensor">
-        <state_interface name="orientation.x" />
-        <state_interface name="orientation.y" />
-        <state_interface name="orientation.z" />
-        <state_interface name="orientation.w" />
-        <state_interface name="angular_velocity.x" />
-        <state_interface name="angular_velocity.y" />
-        <state_interface name="angular_velocity.z" />
-        <state_interface name="linear_acceleration.x" />
-        <state_interface name="linear_acceleration.y" />
-        <state_interface name="linear_acceleration.z" />
-      </sensor> -->
-    </ros2_control>
-    <gazebo>
-      <plugin name="gazebo_ros2_control" filename="libgazebo_ros2_control.so">
-        <ros>
-          <namespace>$(arg model_name)</namespace>
-          <remapping>/$(arg model_name)/joint_states:=/joint_state_broadcaster/joint_states</remapping>
-        </ros>
-        <parameters>$(find sim_models)/models/${model_class}/${model}/config/$(arg gazebo_version)/${model}_controllers.yaml</parameters>
-      </plugin>
-    </gazebo>
-  </xacro:if>
-  <xacro:if value="${gazebo_version == 'latest'}">
-    <ros2_control name="GazeboSimSystem" type="system">
-      <hardware>
-        <plugin>gz_ros2_control/GazeboSimSystem</plugin>
-      </hardware>
-      <joint name="left_wheel_joint">
-        <command_interface name="velocity"/>
-        <state_interface name="position" />
-        <state_interface name="velocity" />
-      </joint>
-      <joint name="right_wheel_joint">
-          <command_interface name="velocity" />
-          <state_interface name="velocity" />
-          <state_interface name="position" />
-      </joint>
-      <!-- <sensor name="imu_sensor">
-        <state_interface name="orientation.x" />
-        <state_interface name="orientation.y" />
-        <state_interface name="orientation.z" />
-        <state_interface name="orientation.w" />
-        <state_interface name="angular_velocity.x" />
-        <state_interface name="angular_velocity.y" />
-        <state_interface name="angular_velocity.z" />
-        <state_interface name="linear_acceleration.x" />
-        <state_interface name="linear_acceleration.y" />
-        <state_interface name="linear_acceleration.z" />
-      </sensor> -->
-    </ros2_control>
-    <gazebo>
-      <plugin filename="gz_ros2_control-system" name="gz_ros2_control::GazeboSimROS2ControlPlugin">
-        <ros>
-          <namespace>/$(arg model_name)</namespace>
-          <remapping>/$(arg model_name)/joint_states:=/joint_state_broadcaster/joint_states</remapping>
-        </ros>
-        <parameters>$(find sim_models)/models/${model_class}/${model}/config/$(arg gazebo_version)/${model}_controllers.yaml</parameters>
-      </plugin>
-    </gazebo>
-  </xacro:if>
+    </joint>
+    <joint name="tray_revolute_joint">
+      <command_interface name="position"/>
+      <state_interface name="velocity" />
+      <state_interface name="position" />
+    </joint>
+    <joint name="tray_prismatic_joint">
+      <command_interface name="position"/>
+      <state_interface name="velocity" />
+      <state_interface name="position" />
+    </joint>
+    <!-- <sensor name="imu_sensor">
+      <state_interface name="orientation.x" />
+      <state_interface name="orientation.y" />
+      <state_interface name="orientation.z" />
+      <state_interface name="orientation.w" />
+      <state_interface name="angular_velocity.x" />
+      <state_interface name="angular_velocity.y" />
+      <state_interface name="angular_velocity.z" />
+      <state_interface name="linear_acceleration.x" />
+      <state_interface name="linear_acceleration.y" />
+      <state_interface name="linear_acceleration.z" />
+    </sensor> -->
+  </ros2_control>
+  <gazebo>
+    <xacro:if value="${gazebo_version == 'classic'}">
+      <xacro:property name="plugin_name" value="gazebo_ros2_control"/>
+      <xacro:property name="plugin_filename" value="libgazebo_ros2_control.so"/>
+    </xacro:if>
+    <xacro:if value="${gazebo_version == 'latest'}">
+      <xacro:property name="plugin_name" value="gz_ros2_control::GazeboSimROS2ControlPlugin"/>
+      <xacro:property name="plugin_filename" value="gz_ros2_control-system"/>
+    </xacro:if>
+    <plugin name="${plugin_name}" filename="${plugin_filename}">
+      <ros>
+        <namespace>$(arg model_name)</namespace>
+        <remapping>/$(arg model_name)/joint_states:=/encoder/joint_states</remapping>
+      </ros>
+      <parameters>$(find sim_models)/models/${model_class}/${model}/config/$(arg gazebo_version)/${model}_controllers.yaml</parameters>
+    </plugin>
+  </gazebo>
 </robot>
