Commit message: creating collisions

File: models/robots/w3_600b/urdf/structure/caster_wheel.xacro (robot description, xacro)
@@ -2,4 +2,8 @@
 <robot xmlns:xacro="http://www.ros.org/wiki/xacro">
     <xacro:macro name="caster_wheel" params="name x y z">
+        <xacro:property name="caster_radius" value="${0.0762/2}"/>
+        <xacro:property name="caster_length" value="0.02413"/>
+        <xacro:property name="collision_offset" value="${caster_length/2}"/>
+        <xacro:property name="caster_z_offset" value="0.001"/>
         <!-- BACK RIGHT CASTER -->
         <link name="caster_wheel_${name}_1">
@@ -17,7 +21,7 @@
             </visual>
             <collision>
-                <origin xyz="0 0 0" rpy="0 0 0"/>
+                <origin xyz="0 0 ${collision_offset + caster_z_offset}" rpy="0 0 0"/>
                 <geometry>
-                    <mesh filename="package://sim_models/models/${model_class}/${model}/meshes/MANIFOLD_SOLID_BREP_6641.stl" scale="0.001 0.001 0.001"/>
+                    <cylinder radius="${caster_radius}" length="${caster_length}"/>
                 </geometry>
             </collision>
@@ -40,7 +44,7 @@
             </visual>
             <collision>
-                <origin xyz="0 0 0" rpy="0 0 0"/>
+                <origin xyz="0 0 -${collision_offset + caster_z_offset}" rpy="0 0 0"/>
                 <geometry>
-                    <mesh filename="package://sim_models/models/${model_class}/${model}/meshes/MANIFOLD_SOLID_BREP_7274.stl" scale="0.001 0.001 0.001"/>
+                    <cylinder radius="${caster_radius}" length="${caster_length}"/>
                 </geometry>
             </collision>

File: models/robots/w3_600b/urdf/structure/tray.xacro (robot description, xacro)
@@ -4,10 +4,10 @@
         <link name="tray">
             <inertial>
-                <origin xyz="0.000045 0.218468 -0.0000000000003836" rpy="0 0 0"/>
+                <origin xyz="0 0 0" rpy="0 0 0"/>
                 <mass value="58.666118"/>
                 <inertia ixx="2.038" ixy="0.000005613643" ixz="-0.000000000000003583" iyx="0.000005613643" iyy="5.914" iyz="-0.00000000000002564" izx="-0.000000000000003583" izy="-0.00000000000002564" izz="3.878"/>
             </inertial>
             <visual>
-                <origin xyz="0 0 0" rpy="0 0 0"/>
+                <origin xyz="0 -0.218468 0" rpy="0 0 0"/>
                 <geometry>
                     <mesh filename="package://sim_models/models/${model_class}/${model}/meshes/tray.stl" scale="0.001 0.001 0.001"/>
@@ -18,5 +18,5 @@
                 <origin xyz="0 0 0" rpy="0 0 0"/>
                 <geometry>
-                    <mesh filename="package://sim_models/models/${model_class}/${model}/meshes/tray.stl" scale="0.001 0.001 0.001"/>
+                    <box size="0.924 0.014 0.650"/>
                 </geometry>
             </collision>
@@ -27,5 +27,5 @@
         <link name="rotating_base_link">
             <inertial>
-                <origin xyz="0.000045 0.218468 -0.0000000000003836" rpy="0 0 0"/>
+                <origin xyz="0 0 0" rpy="0 0 0"/>
                 <mass value="58.666118"/>
                 <inertia ixx="2.038" ixy="0.000005613643" ixz="-0.000000000000003583" iyx="0.000005613643" iyy="5.914" iyz="-0.00000000000002564" izx="-0.000000000000003583" izy="-0.00000000000002564" izz="3.878"/>
@@ -35,5 +35,5 @@
             <parent link="base_link"/>
             <child link="rotating_base_link"/>
-            <origin xyz="0 0 0" rpy="0 0 0"/>
+            <origin xyz="0 0.218468 0" rpy="0 0 0"/>
             <axis xyz="0 1 0"/>
             <limit effort="5886" velocity="${300*(3.14/180)}" lower="-6.28" upper="6.28"/>

File: models/robots/w3_600b/urdf/structure/wheel.xacro (robot description, xacro)
@@ -2,4 +2,6 @@
 <robot xmlns:xacro="http://www.ros.org/wiki/xacro">
     <xacro:macro name="wheel" params="name x y z">
+        <xacro:property name="wheel_radius" value="${0.165/2}"/>
+        <xacro:property name="wheel_length" value="0.046"/>
         <link name="${name}_wheel">
             <inertial>
@@ -23,7 +25,7 @@
             </visual>
             <collision>
-                <origin xyz="0 0 ${wheel_z_offset}" rpy="0 0 0"/>
+                <origin xyz="0 0 -${wheel_length/2}" rpy="0 0 0"/>
                 <geometry>
-                    <mesh filename="package://sim_models/models/${model_class}/${model}/meshes/${name}_wheel.stl" scale="0.001 0.001 0.001"/>
+                    <cylinder radius="${wheel_radius}" length="${wheel_length}"/>
                 </geometry>
             </collision>

File: models/robots/w3_600b/urdf/w3_600b.xacro (robot description, xacro)
@@ -44,5 +44,5 @@
       <origin xyz="0 0 0" rpy="0 0 0"/>
       <geometry>
-        <mesh filename="package://sim_models/models/${model_class}/${model}/meshes/base_link_v2.stl" scale="0.001 0.001 0.001"/>
+        <mesh filename="package://sim_models/models/${model_class}/${model}/meshes/base.stl" scale="0.001 0.001 0.001"/>
       </geometry>
     </collision>
@@ -60,8 +60,8 @@
   <xacro:caster_wheel name="fr" x="0.335" y="0.0131" z="0.157"/>
   <xacro:caster_wheel name="fl" x="0.335" y="0.0131" z="-0.197"/>
-  <!-- <xacro:camera name="down"/>
+  <xacro:camera name="down"/>
   <xacro:camera name="up"/>
   <xacro:lidar name="front"/>
-  <xacro:lidar name="back"/> -->
+  <xacro:lidar name="back"/>
   <xacro:imu_gazebo/>
   <xacro:wheel name="left" x="0" y="0.0575" z="-0.131553"/>
